File: Hardware/eagle/main_board.brd (EAGLE design)
At the start: 101.3 x 83.8 mm, 59 parts, among them IC1 INA238AIDGST, IC10 INA238AIDGST, IC11 INA238AIDGST, IC2 INA238AIDGST, IC3 INA238AIDGST, IC5 LT1129MPST-3.3#PBF, IC7 ESP-WROOM-32__16MB_, IC8 AVR128DB48-I_PT, IC9 INA238AIDGST, M1 1751248, M2 1751248, M3 1751248, M4 1751248, M5 1751248, X1 1751248

Commit message: main_board.brd - Layout
Parts:
- added C7: (no value), rcl:C0603
- added IC4: R-78E3.3-1.0, SamacSys_Parts:R78E3310
- added IC6: INA238AIDGST, SamacSys_Parts:SOP50P490X110-10N
- added R5: 0R0, rcl:R0603
- added R6: Y08500R10000F9R, SamacSys_Parts:Y08500R10000F9R
- moved C11 66.4 mm to (41.3, 70.2), turned to 180 degrees
- moved C4 62.1 mm to (41.3, 72.4), turned to 180 degrees
- moved C3 59.2 mm to (37.8, 72.4), turned to 0 degrees
- moved C14 48.1 mm to (19.1, 79.4), flipped to the bottom, turned to 90 degrees
- moved C8 45.3 mm to (22.9, 70.8), flipped to the bottom, turned to 0 degrees
- moved C15 44.9 mm to (31.8, 79.4), flipped to the bottom, turned to 90 degrees
- moved C23 44.7 mm to (21.6, 38.7), flipped to the bottom, turned to 0 degrees
- moved C9 43.8 mm to (21.6, 64.5), flipped to the bottom, turned to 0 degrees
- moved R3 42.4 mm to (41.3, 67.9), turned to 180 degrees
- moved C6 34.0 mm to (21.6, 15.9), flipped to the bottom, turned to 0 degrees
- moved C5 31.8 mm to (21.6, 8.26), flipped to the bottom, turned to 0 degrees
- moved C22 31.5 mm to (21.6, 23.5), flipped to the bottom, turned to 0 degrees
- moved C24 31.4 mm to (21.6, 45.7), flipped to the bottom, turned to 0 degrees
- moved C10 28.1 mm to (21.6, 31.1), flipped to the bottom, turned to 0 degrees
- moved SJ1 17.2 mm to (30.2, 70.5)
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Connections:
- removed net +24V1: BATT.1, IC1.8, IC2.8, IC3.8, R1.1, R10.1, R2.1, X1.1
- removed net +24V3: IC11.8, R16.1
- removed net N$35: C23.1, C24.1, IC11.6
- removed net N$36: C10.1, C22.1, IC10.6, IC9.6
- new net N$11: IC6.10, R6.3
- new net N$12: BATT.1, R6.2
- new net N$5: C13.1, C15.1, IC4.3, R5.1
- new net N$9: IC6.9, R6.4
- net +24V: now also IC4.1
- net +24V2: now also IC1.8, IC11.8, IC2.8, IC3.8, IC6.8, R1.1, R10.1, R16.1, R2.1, R6.1, X1.1
- net +3V3: now also C10.1, C22.1, C23.1, C24.1, C7.1, IC10.6, IC11.1, IC11.6, IC6.1, IC6.6, IC9.6; no longer U$3.P$5
- net +5V: now also R5.2; no longer C13.1, C15.1
- net GND: now also C7.2, IC10.1, IC11.2, IC6.7, IC9.1; no longer U$3.P$1
- net GNDA: now also IC4.2
- net I2C_0_SCL: now also IC10.2, IC6.5; no longer I2C_IO_1.2, I2C_IO_2.2, U$3.P$3
- net I2C_0_SDA: now also IC6.2, IC6.4, IC9.2; no longer I2C_IO_1.3, I2C_IO_2.3, U$3.P$4
- net I2C_1_SCL: now also I2C_IO_1.2, I2C_IO_2.2
- net I2C_1_SDA: now also I2C_IO_1.3, I2C_IO_2.3
Routing:
- net +24V2: track 0.00 -> 130.0 mm, vias 0 -> 6
- net I2C_0_SDA: track 0.00 -> 88.3 mm, vias 0 -> 7
- net I2C_0_SCL: track 0.00 -> 82.9 mm, vias 0 -> 7
- net +3V3: track 0.00 -> 65.6 mm
- net N$12: track 0.00 -> 9.79 mm
- net N$27: track 0.00 -> 8.91 mm, vias 0 -> 1
- net N$33: track 0.00 -> 8.91 mm, vias 0 -> 1
- net N$6: track 0.00 -> 8.91 mm, vias 0 -> 1
- net N$25: track 0.00 -> 8.91 mm, vias 0 -> 1
- net N$2: track 0.00 -> 8.00 mm
- net N$3: track 0.00 -> 8.00 mm
- net N$32: track 0.00 -> 7.98 mm
- net N$22: track 0.00 -> 7.98 mm
- net N$1: track 0.00 -> 7.98 mm
- net N$9: track 0.00 -> 7.64 mm, vias 0 -> 1
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
Commit message: Layout
Parts:
- removed I2C_IO_1, I2C_IO_2: (no value), con-lstb:MA04-1
- removed LED: (no value), con-ml:ML6
- removed SV2, SV3: (no value), con-lstb:MA04-2
- added C20, C21, C38: 5p6, rcl:C0603
- added C25, C33: 4.7µ, rcl:C0603
- added C26, C27, C28, C29, C30, C31, C32, C34, C35, C36, C39, C40, C41, C42, C43, C44, C45, C46: 100n, rcl:C0603
- added C37: 1n, rcl:C0603
- added C47, C48: (no value), rcl:C0603
- added D1: BAT760-7, SamacSys_Parts:SOD2513X120N
- added D2: PRTR5V0U2AX,215, SamacSys_Parts:PESD2ETHAXR
- added IC12: ATSAME70N21B-AN, SamacSys_Parts:QFP50P1600X1600X160-100N
- added J1: 47346-0001, SamacSys_Parts:47346-0001
- added J2, J3: B06B-XASK-1, SamacSys_Parts:SHDR6W60P0X250_1X6_1750X640X88
- added J4, J5, J6: B03B-XASK-1, SamacSys_Parts:SHDR3W60P0X250_1X3_1000X640X88
- added J7, J8: B05B-XASK-1, SamacSys_Parts:SHDR5W60P0X250_1X5_1500X640X88
- added R17, R7, R8, R9: 47k, rcl:R0603
- added R18, R19: (no value), rcl:R0603
- added SWD: 3220-10-0300-00, SamacSys_Parts:3220-10-0300-00
- added Y1: 32.768kHz, microbuilder:CRYSTAL_4.9X1.8
- moved C2 55.1 mm to (94.0, 56.2), flipped to the bottom, turned to 270 degrees
- moved C1 51.3 mm to (92.4, 56.2), flipped to the bottom, turned to 270 degrees
- moved MOD4 37.3 mm to (92.7, 36.2), turned to 180 degrees
- moved R14 21.7 mm to (66.0, 6.35), flipped to the bottom
- moved R11 21.1 mm to (47.6, 6.35), flipped to the bottom
- moved C16 18.8 mm to (47.6, 10.5), flipped to the bottom
- moved MOD2 17.4 mm to (75.2, 36.2)
- moved IC7 17.2 mm to (79.4, 75.6)
- moved C19 16.9 mm to (66.0, 10.5), flipped to the bottom
- moved R12 13.9 mm to (50.2, 6.35), flipped to the bottom
- moved C17 13.7 mm to (50.2, 10.5), flipped to the bottom
- moved MOD1 13.5 mm to (78.4, 17.5), turned to 180 degrees
- moved GPS 13.1 mm to (96.5, 58.7)
- moved R13 11.2 mm to (52.7, 6.35), flipped to the bottom
- moved C18 9.14 mm to (52.7, 10.5), flipped to the bottom
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Connections:
- removed net UART_RXD: GPS.2
- removed net UART_TXD: GPS.1
- removed net WS2812B_OUT: LED.3, LED.4
- new net ADC_REGEN_SENS: J6.2
- new net DISP_CS: IC12.48
- new net DISP_DC: IC12.44
- new net DISP_RS: IC12.42
- new net GPS_PPS: IC12.34
- new net ML_MON_CUR: IC12.14
- new net ML_NFAULT: IC12.20
- new net ML_PHASE: IC12.21
- new net MOT_EN: IC12.80
- new net MOT_MON_CUR: IC12.16
- new net MOT_NFAULT: IC12.77
- new net MOT_NSLEEP: IC12.79
- new net MOT_PHASE: IC12.78
- new net MR_MON_CUR: IC12.15
- new net MR_NFAULT: IC12.1
- new net MR_PHASE: IC12.2
- new net N$13: C37.1, D1.2, D2.4, J1.1
- new net N$16: IC12.60, R7.2
- new net N$17: J2.5, R13.1
- new net N$18: J2.3, R11.1
- new net N$35: C47.1, R18.2
- new net N$36: C19.1, R14.2
- new net PA09_UART_RXD_0: IC12.54
- new net PA10_UART_TXD_0: IC12.46
- new net PA20_PERIMETER_SENDER: IC12.13
- new net PA21_USB_N: D2.3, IC12.94, J1.2
- new net PA22_USB_P: D2.2, IC12.95, J1.3
- new net PA7_XIN32: C20.1, IC12.24, Y1.1
- new net PA8_XOUT32: C21.1, IC12.25, Y1.2
- new net PB01_SPI_4_SCK: IC12.47
- new net PB10_SPI_4_MOSI: IC12.43
- new net PB11_SPI_4_MISO: IC12.45
- new net PB6_SWDIO_TMS: IC12.57, R8.1, SWD.2
- new net PB7_SWCLK_TCK: IC12.63, R9.1, SWD.4
- new net PD25_UART_RXD_2: IC12.35
- new net PD26_UART_TXD_2: IC12.36
- new net SENSOR_SCL: IC12.55
- new net SENSOR_SDA: IC12.64
- new net TARGET_RESET: C38.1, IC12.58, R17.1, SWD.10
- new net TOUCH_CS: IC12.50
- new net TOUCH_IRQ: IC12.49
- new net VCCINT: C33.1, C34.1, C35.1, C36.1, C39.1, C40.1, C41.1, C42.1, C43.1, C44.1, IC12.18, IC12.22, IC12.39, IC12.4, IC12.76, IC12.86, IC12.96
- new net WS2812B_1_OUT: J4.2
- new net WS2812B_2_OUT: J5.2
- net +3V3: now also C25.1, C26.1, C27.1, C28.1, C29.1, C30.1, C31.1, C32.1, C45.1, C46.1, IC12.19, IC12.28, IC12.5, IC12.68, IC12.81, IC12.9, IC12.90, IC12.93, J2.2, J3.2, J7.2, J8.2, R17.2, R8.2, R9.2, SWD.1; no longer I2C_IO_1.1, I2C_IO_2.1, SV2.5, SV2.6, SV3.5, SV3.6
- net +5V: now also D1.1, J2.1, J3.1, J4.1, J5.1, J6.1, J7.1, J8.1; no longer LED.1, LED.2, SV2.7, SV2.8, SV3.7, SV3.8
- net GND: now also C20.2, C21.2, C25.2, C26.2, C27.2, C28.2, C29.2, C30.2, C31.2, C32.2, C33.2, C34.2, C35.2, C36.2, C37.2, C38.2, C39.2, C40.2, C41.2, C42.2, C43.2, C44.2, C45.2, C46.2, C47.2, C48.2, D2.1, IC12.10, IC12.29, IC12.3, IC12.6, IC12.67, IC12.7, IC12.8, J1.5, J2.6, J3.6, J4.3, J5.3, J6.3, J7.5, J8.5, R7.1, SWD.3, SWD.5, SWD.9; no longer I2C_IO_1.4, I2C_IO_2.4, LED.5, LED.6, SV2.1, SV2.2, SV3.1, SV3.2
- net I2C_0_SCL: now also J7.3, J8.3; no longer IC1.5, IC10.2, IC10.5, IC11.5, IC2.5, IC3.5, IC6.5, IC9.5, U$3.P$9
- net I2C_0_SDA: now also J7.4, J8.4; no longer IC1.4, IC10.4, IC11.4, IC2.4, IC3.4, IC6.2, IC6.4, IC9.2, IC9.4, U$3.P$10
- net I2C_1_SCL: now also IC1.5, IC10.2, IC10.5, IC11.5, IC2.5, IC3.5, IC6.5, IC9.5, U$3.P$9; no longer I2C_IO_1.2, I2C_IO_2.2
- net I2C_1_SDA: now also IC1.4, IC10.4, IC11.4, IC2.4, IC3.4, IC6.2, IC6.4, IC9.2, IC9.4, U$3.P$10; no longer I2C_IO_1.3, I2C_IO_2.3
- net N$14: now also C18.1, R13.2; no longer C17.1, R11.2
- net N$15: now also J2.4; no longer SV2.4
- net N$19: now also C17.1, R12.2; no longer R11.1, SV2.3
- net N$23: now also R11.2; no longer R12.2
- net N$24: now also J3.4, R18.1; no longer C19.1, R13.2
- net N$26: now also J3.5, R19.1; no longer R14.1, SV3.4
- net N$28: now also J3.3, R14.1; no longer R13.1, SV3.3
- net N$30: now also C48.1, R19.2; no longer C18.1, R14.2
- net UART_0_RXD: now also GPS.2
- net UART_0_TXD: now also GPS.1
Routing:
- net I2C_0_SDA: track 88.3 -> 0.00 mm, vias 7 -> 0
- net I2C_0_SCL: track 82.9 -> 0.00 mm, vias 7 -> 0
- net I2C_1_SCL: track 0.00 -> 79.0 mm, vias 0 -> 7
- net I2C_1_SDA: track 0.00 -> 71.4 mm, vias 0 -> 7

Commit message: Layout
Parts:
- removed C20, C21: 5p6, rcl:C0603
- removed C25, C33: 4.7µ, rcl:C0603
- removed C26, C27, C28, C29, C30, C31, C32, C34, C35, C36, C39, C40, C41, C42, C43, C44, C45, C46: 100n, rcl:C0603
- removed C37: 1n, rcl:C0603
- removed D1: BAT760-7, SamacSys_Parts:SOD2513X120N
- removed D2: PRTR5V0U2AX,215, SamacSys_Parts:PESD2ETHAXR
- removed IC12: ATSAME70N21B-AN, SamacSys_Parts:QFP50P1600X1600X160-100N
- removed J1: 47346-0001, SamacSys_Parts:47346-0001
- removed R9: 47k, rcl:R0603
- removed SWD: 3220-10-0300-00, SamacSys_Parts:3220-10-0300-00
- removed U$3: PCA9685_BREAKOUT_ONLY_I2C, SamacSys_Parts:PCA9685_BREAKOUT_ONLY_I2C
- removed Y1: 32.768kHz, microbuilder:CRYSTAL_4.9X1.8
- added C49: (no value), rcl:C0603
- added IC13: PCA9685PW, SamacSys_Parts:SOP65P640X110-28N
- added PROG: 3220-10-0300-00, SamacSys_Parts:3220-10-0300-00
- added R25: (no value), rcl:R0603
- added SV1, SV2: (no value), con-lstb:MA10-1
- R7: value 47k -> 33R
- moved C38 125.7 mm to (55.2, 64.1)
- moved R7 124.9 mm to (55.2, 66.7)
- moved R8 124.8 mm to (65.7, 64.5), turned to 270 degrees
- moved R17 122.5 mm to (55.2, 62.5)
Connections:
- removed net DISP_CS: IC12.48
- removed net DISP_DC: IC12.44
- removed net DISP_RS: IC12.42
- removed net GPS_PPS: IC12.34
- removed net ML_MON_CUR: IC12.14
- removed net ML_NFAULT: IC12.20
- removed net ML_PHASE: IC12.21
- removed net MOT_EN: IC12.80
- removed net MOT_MON_CUR: IC12.16
- removed net MOT_NFAULT: IC12.77
- removed net MOT_NSLEEP: IC12.79
- removed net MOT_PHASE: IC12.78
- removed net MR_MON_CUR: IC12.15
- removed net MR_NFAULT: IC12.1
- removed net MR_PHASE: IC12.2
- removed net PA09_UART_RXD_0: IC12.54
- removed net PA10_UART_TXD_0: IC12.46
- removed net PA20_PERIMETER_SENDER: IC12.13
- removed net PA21_USB_N: D2.3, IC12.94, J1.2
- removed net PA22_USB_P: D2.2, IC12.95, J1.3
- removed net PA7_XIN32: C20.1, IC12.24, Y1.1
- removed net PA8_XOUT32: C21.1, IC12.25, Y1.2
- removed net PB01_SPI_4_SCK: IC12.47
- removed net PB10_SPI_4_MOSI: IC12.43
- removed net PB11_SPI_4_MISO: IC12.45
- removed net PB6_SWDIO_TMS: IC12.57, R8.1, SWD.2
- removed net PB7_SWCLK_TCK: IC12.63, R9.1, SWD.4
- removed net PD25_UART_RXD_2: IC12.35
- removed net PD26_UART_TXD_2: IC12.36
- removed net SENSOR_SCL: IC12.55
- removed net SENSOR_SDA: IC12.64
- removed net SPI_1_CS: IC8.13
- removed net SPI_1_MISO: IC8.11
- removed net SPI_1_MOSI: IC8.10
- removed net SPI_1_SCK: IC8.12
- removed net TARGET_RESET: C38.1, IC12.58, R17.1, SWD.10
- removed net TOUCH_CS: IC12.50
- removed net TOUCH_IRQ: IC12.49
- removed net UART_1_RXD: IC8.17
- removed net UART_1_TXD: IC8.16
- removed net VCCINT: C33.1, C34.1, C35.1, C36.1, C39.1, C40.1, C41.1, C42.1, C43.1, C44.1, IC12.18, IC12.22, IC12.39, IC12.4, IC12.76, IC12.86, IC12.96
- new net AIN_00: C16.1, IC8.20, R11.2
- new net AIN_01: C17.1, IC8.21, R12.2
- new net AIN_02: C18.1, IC8.22, R13.2
- new net AIN_03: C19.1, IC8.23, R14.2
- new net AIN_04: C47.1, IC8.24, R18.2
- new net AIN_05: C48.1, IC8.25, R19.2
- new net AIN_06: C49.1, IC8.26, R25.2
- new net CURR_ALERT_CHRG: IC6.3, IC8.4
- new net CURR_ALERT_M1: IC1.3, IC8.11
- new net CURR_ALERT_M2: IC2.3, IC8.10
- new net CURR_ALERT_M3: IC8.9, IC9.3
- new net CURR_ALERT_M4: IC10.3, IC8.8
- new net CURR_ALERT_M5: IC11.3, IC8.5
- new net CURR_ALERT_SYS: IC3.3, IC8.3
- new net N$37: IC8.48
- new net N$38: IC13.11, SV1.7
- new net N$40: IC13.12, SV1.8
- new net N$41: IC13.13, SV1.9
- new net N$42: IC13.16, SV2.3
- new net N$43: IC13.17, SV2.4
- new net N$44: IC13.18, SV2.5
- new net N$45: IC13.19, SV2.6
- new net N$46: IC13.20, SV2.7
- new net N$47: IC13.21, SV2.8
- new net N$48: IC13.22, SV2.9
- new net PWM_PCA9685_OE: IC13.23, IC8.12
- new net UART_2_RXD: IC8.39
- new net UART_2_TXD: IC8.38
- net +3V3: now also IC13.28, PROG.4, SV1.1, SV2.1; no longer C25.1, C26.1, C27.1, C28.1, C29.1, C30.1, C31.1, C32.1, C45.1, C46.1, IC12.19, IC12.28, IC12.5, IC12.68, IC12.81, IC12.9, IC12.90, IC12.93, R9.2, SWD.1, U$3.P$11
- net +5V: no longer D1.1
- net /RESET: now also C38.1, R17.1, R7.1
- net ADC_REGEN_SENS: now also R25.1
- net GND: now also C49.2, IC13.14, PROG.2, PROG.9, SV1.10, SV2.10; no longer C20.2, C21.2, C25.2, C26.2, C27.2, C28.2, C29.2, C30.2, C31.2, C32.2, C33.2, C34.2, C35.2, C36.2, C37.2, C39.2, C40.2, C41.2, C42.2, C43.2, C44.2, C45.2, C46.2, D2.1, IC12.10, IC12.29, IC12.3, IC12.6, IC12.67, IC12.7, IC12.8, J1.5, R7.1, SWD.3, SWD.5, SWD.9, U$3.P$7
- net I2C_1_SCL: now also IC13.26; no longer U$3.P$9
- net I2C_1_SDA: now also IC13.27; no longer U$3.P$10
- net N$13: now also PROG.3, R8.1; no longer C37.1, D1.2, D2.4, J1.1
- net N$14: now also IC13.15, SV2.2; no longer C18.1, R13.2
- net N$16: now also PROG.6; no longer IC12.60
- net N$19: now also IC13.6, SV1.2; no longer C17.1, R12.2
- net N$23: now also IC13.7, SV1.3; no longer C16.1, R11.2
- net N$30: now also IC13.8, SV1.4; no longer C48.1, R19.2
- net N$35: now also IC13.9, SV1.5; no longer C47.1, R18.2
- net N$36: now also IC13.10, SV1.6; no longer C19.1, R14.2
- net SPI_0_CS: now also IC8.33; no longer IC8.3
- net SPI_0_MISO: now also IC8.31; no longer IC8.1
- net SPI_0_MOSI: now also IC8.30; no longer IC8.48
- net SPI_0_SCK: now also IC8.32; no longer IC8.2
Routing:
- net I2C_0_SDA: track 0.00 -> 87.0 mm, vias 0 -> 1
- net I2C_0_SCL: track 0.00 -> 85.7 mm, vias 0 -> 1
- net CURR_ALERT_SYS: track 0.00 -> 50.1 mm, vias 0 -> 1
- net CURR_ALERT_M1: track 0.00 -> 49.4 mm, vias 0 -> 1
- net UART_0_RXD: track 0.00 -> 46.8 mm
- net UART_0_TXD: track 0.00 -> 44.8 mm
- net CURR_ALERT_M2: track 0.00 -> 43.0 mm, vias 0 -> 1
- net CURR_ALERT_M3: track 0.00 -> 36.5 mm, vias 0 -> 1
- net I2C_1_SDA: track 71.4 -> 107.8 mm, vias 7 -> 9
- net CURR_ALERT_CHRG: track 0.00 -> 36.1 mm, vias 0 -> 1
- net +3V3: track 65.6 -> 95.6 mm
- net CURR_ALERT_M4: track 0.00 -> 29.7 mm, vias 0 -> 1
- net +24V: track 0.00 -> 28.2 mm, vias 0 -> 1
- net CURR_ALERT_M5: track 0.00 -> 27.2 mm, vias 0 -> 1
- net PWM_PCA9685_OE: track 0.00 -> 23.3 mm
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