File: Hardware/eagle/main_board.sch (EAGLE design)
At the start: 59 parts, among them IC1 INA238AIDGST, IC10 INA238AIDGST, IC11 INA238AIDGST, IC2 INA238AIDGST, IC3 INA238AIDGST, IC5 LT1129MPST-3.3#PBF, IC7 ESP-WROOM-32__16MB_, IC8 AVR128DB48-I_PT, IC9 INA238AIDGST, M1 1751248, M2 1751248, M3 1751248, M4 1751248, M5 1751248, X1 1751248

Commit message: main_board.brd - Layout
Parts:
- added C7: (no value), rcl:C-EUC0603
- added IC4: R-78E3.3-1.0, SamacSys_Parts:R-78E3.3-1.0
- added IC6: INA238AIDGST, SamacSys_Parts:INA238AIDGST
- added R5: 0R0, rcl:R-EU_R0603
- added R6: Y08500R10000F9R, SamacSys_Parts:Y08500R10000F9R
Connections:
- removed net +24V1: BATT-1.K, IC1.VBUS, IC2.VBUS, IC3.VBUS, R1.1, R10.1, R2.1, X1-1.K
- removed net +24V3: IC11.VBUS, R16.1
- removed net N$35: C23.1, C24.1, IC11.VS
- removed net N$36: C10.1, C22.1, IC10.VS, IC9.VS
- new net N$11: IC6.IN+, R6.3
- new net N$12: BATT-1.K, R6.2
- new net N$5: C13.1, C15.1, IC4.+VOUT, R5.1
- new net N$9: IC6.IN-, R6.4
- net +24V: now also IC4.+VIN
- net +24V2: now also IC1.VBUS, IC11.VBUS, IC2.VBUS, IC3.VBUS, IC6.VBUS, R1.1, R10.1, R16.1, R2.1, R6.1, X1-1.K
- net +3V3: now also C10.1, C22.1, C23.1, C24.1, C7.1, IC10.VS, IC11.A1, IC11.VS, IC6.A1, IC6.VS, IC9.VS; no longer U$3.VCC
- net +5V: now also R5.2; no longer C13.1, C15.1
- net GND: now also C7.2, IC10.A1, IC11.A0, IC6.GND, IC9.A1; no longer U$3.GND
- net GNDA: now also IC4.GND
- net I2C_0_SCL: now also IC10.A0, IC6.SCL; no longer I2C_IO_1.2, I2C_IO_2.2, U$3.SCL
- net I2C_0_SDA: now also IC6.A0, IC6.SDA, IC9.A0; no longer I2C_IO_1.3, I2C_IO_2.3, U$3.SDA
- net I2C_1_SCL: now also I2C_IO_1.2, I2C_IO_2.2
- net I2C_1_SDA: now also I2C_IO_1.3, I2C_IO_2.3
Other:
- note removed: "U = 5.1034V"
- moved on the sheet: BATT-1, BATT-2, C11, C13, C15, C3, C4, IC5, R3, SJ1

Commit message: Layout
Parts:
- removed I2C_IO_1, I2C_IO_2: (no value), con-lstb:MA04-1
- removed LED: (no value), con-ml:ML6
- removed SV2, SV3: (no value), con-lstb:MA04-2
- added C20, C21, C38: 5p6, rcl:C-EUC0603
- added C25, C33: 4.7µ, rcl:C-EUC0603
- added C26, C27, C28, C29, C30, C31, C32, C34, C35, C36, C39, C40, C41, C42, C43, C44, C45, C46: 100n, rcl:C-EUC0603
- added C37: 1n, rcl:C-EUC0603
- added C47, C48: (no value), rcl:C-EUC0603
- added D1: BAT760-7, SamacSys_Parts:BAT760-7
- added D2: PRTR5V0U2AX,215, SamacSys_Parts:PRTR5V0U2AX,215
- added IC12: ATSAME70N21B-AN, SamacSys_Parts:ATSAME70N21B-AN
- added J1: 47346-0001, SamacSys_Parts:47346-0001
- added J2, J3: B06B-XASK-1, SamacSys_Parts:B06B-XASK-1
- added J4, J5, J6: B03B-XASK-1, SamacSys_Parts:B03B-XASK-1
- added J7, J8: B05B-XASK-1, SamacSys_Parts:B05B-XASK-1
- added R17, R7, R8, R9: 47k, rcl:R-EU_R0603
- added R18, R19: (no value), rcl:R-EU_R0603
- added SWD: 3220-10-0300-00, SamacSys_Parts:3220-10-0300-00
- added Y1: 32.768kHz, microbuilder:CRYSTALTHIN32K
Connections:
- removed net UART_RXD: GPS.2
- removed net UART_TXD: GPS.1
- removed net WS2812B_OUT: LED.3, LED.4
- new net ADC_REGEN_SENS: J6.2
- new net DISP_CS: IC12.PA12
- new net DISP_DC: IC12.PA11
- new net DISP_RS: IC12.PA26
- new net GPS_PPS: IC12.PA14
- new net ML_MON_CUR: IC12.PA19
- new net ML_NFAULT: IC12.PB3
- new net ML_PHASE: IC12.PA21
- new net MOT_EN: IC12.PD8
- new net MOT_MON_CUR: IC12.PA17
- new net MOT_NFAULT: IC12.PB5
- new net MOT_NSLEEP: IC12.PA28
- new net MOT_PHASE: IC12.PD9
- new net MR_MON_CUR: IC12.PA18
- new net MR_NFAULT: IC12.PD0
- new net MR_PHASE: IC12.PD31
- new net N$13: C37.1, D1.A, D2.VCC, J1.VBUS
- new net N$16: IC12.TST, R7.2
- new net N$17: J2.5, R13.1
- new net N$18: J2.3, R11.1
- new net N$35: C47.1, R18.2
- new net N$36: C19.1, R14.2
- new net PA09_UART_RXD_0: IC12.PA9
- new net PA10_UART_TXD_0: IC12.PA10
- new net PA20_PERIMETER_SENDER: IC12.PA20
- new net PA21_USB_N: D2.I/O_2, IC12.HSDM, J1.D-
- new net PA22_USB_P: D2.I/O_1, IC12.HSDP, J1.D+
- new net PA7_XIN32: C20.1, IC12.PA7, Y1.1
- new net PA8_XOUT32: C21.1, IC12.PA8, Y1.2
- new net PB01_SPI_4_SCK: IC12.PD19
- new net PB10_SPI_4_MOSI: IC12.PD21
- new net PB11_SPI_4_MISO: IC12.PD20
- new net PB6_SWDIO_TMS: IC12.PB6, R8.1, SWD.2
- new net PB7_SWCLK_TCK: IC12.PB7, R9.1, SWD.4
- new net PD25_UART_RXD_2: IC12.PD25
- new net PD26_UART_TXD_2: IC12.PD26
- new net SENSOR_SCL: IC12.PA4
- new net SENSOR_SDA: IC12.PA3
- new net TARGET_RESET: C38.1, IC12.NRST, R17.1, SWD.10
- new net TOUCH_CS: IC12.PA27
- new net TOUCH_IRQ: IC12.PD18
- new net VCCINT: C33.1, C34.1, C35.1, C36.1, C39.1, C40.1, C41.1, C42.1, C43.1, C44.1, IC12.VDDCORE_1, IC12.VDDCORE_2, IC12.VDDCORE_3, IC12.VDDCORE_4, IC12.VDDOUT, IC12.VDDPLL, IC12.VDDUTMIC
- new net WS2812B_1_OUT: J4.2
- new net WS2812B_2_OUT: J5.2
- net +3V3: now also C25.1, C26.1, C27.1, C28.1, C29.1, C30.1, C31.1, C32.1, C45.1, C46.1, IC12.VDDIN, IC12.VDDIO_1, IC12.VDDIO_2, IC12.VDDIO_3, IC12.VDDIO_4, IC12.VDDPLLUSB, IC12.VDDUTMII, IC12.VREFP, J2.2, J3.2, J7.2, J8.2, R17.2, R8.2, R9.2, SWD.1; no longer I2C_IO_1.1, I2C_IO_2.1, SV2.5, SV2.6, SV3.5, SV3.6
- net +5V: now also D1.K, J2.1, J3.1, J4.1, J5.1, J6.1, J7.1, J8.1; no longer LED.1, LED.2, SV2.7, SV2.8, SV3.7, SV3.8
- net GND: now also C20.2, C21.2, C25.2, C26.2, C27.2, C28.2, C29.2, C30.2, C31.2, C32.2, C33.2, C34.2, C35.2, C36.2, C37.2, C38.2, C39.2, C40.2, C41.2, C42.2, C43.2, C44.2, C45.2, C46.2, C47.2, C48.2, D2.GND, IC12.GND_1, IC12.GND_2, IC12.GND_3, IC12.GND_4, IC12.GND_5, IC12.GND_6, IC12.VREFN, J1.GND, J2.6, J3.6, J4.3, J5.3, J6.3, J7.5, J8.5, R7.1, SWD.3, SWD.5, SWD.9; no longer I2C_IO_1.4, I2C_IO_2.4, LED.5, LED.6, SV2.1, SV2.2, SV3.1, SV3.2
- net I2C_0_SCL: now also J7.3, J8.3; no longer IC1.SCL, IC10.A0, IC10.SCL, IC11.SCL, IC2.SCL, IC3.SCL, IC6.SCL, IC9.SCL, U$3.SCL.
- net I2C_0_SDA: now also J7.4, J8.4; no longer IC1.SDA, IC10.SDA, IC11.SDA, IC2.SDA, IC3.SDA, IC6.A0, IC6.SDA, IC9.A0, IC9.SDA, U$3.SDA.
- net I2C_1_SCL: now also IC1.SCL, IC10.A0, IC10.SCL, IC11.SCL, IC2.SCL, IC3.SCL, IC6.SCL, IC9.SCL, U$3.SCL.; no longer I2C_IO_1.2, I2C_IO_2.2
- net I2C_1_SDA: now also IC1.SDA, IC10.SDA, IC11.SDA, IC2.SDA, IC3.SDA, IC6.A0, IC6.SDA, IC9.A0, IC9.SDA, U$3.SDA.; no longer I2C_IO_1.3, I2C_IO_2.3
- net N$14: now also C18.1, R13.2; no longer C17.1, R11.2
- net N$15: now also J2.4; no longer SV2.4
- net N$19: now also C17.1, R12.2; no longer R11.1, SV2.3
- net N$23: now also R11.2; no longer R12.2
- net N$24: now also J3.4, R18.1; no longer C19.1, R13.2
- net N$26: now also J3.5, R19.1; no longer R14.1, SV3.4
- net N$28: now also J3.3, R14.1; no longer R13.1, SV3.3
- net N$30: now also C48.1, R19.2; no longer C18.1, R14.2
- net UART_0_RXD: now also GPS.2
- net UART_0_TXD: now also GPS.1
Other:
- moved on the sheet: C16, C17, C18, C19, R11, R12, R13, R14

Commit message: Layout
Parts:
- removed C20, C21: 5p6, rcl:C-EUC0603
- removed C25, C33: 4.7µ, rcl:C-EUC0603
- removed C26, C27, C28, C29, C30, C31, C32, C34, C35, C36, C39, C40, C41, C42, C43, C44, C45, C46: 100n, rcl:C-EUC0603
- removed C37: 1n, rcl:C-EUC0603
- removed D1: BAT760-7, SamacSys_Parts:BAT760-7
- removed D2: PRTR5V0U2AX,215, SamacSys_Parts:PRTR5V0U2AX,215
- removed IC12: ATSAME70N21B-AN, SamacSys_Parts:ATSAME70N21B-AN
- removed J1: 47346-0001, SamacSys_Parts:47346-0001
- removed R9: 47k, rcl:R-EU_R0603
- removed SWD: 3220-10-0300-00, SamacSys_Parts:3220-10-0300-00
- removed U$3: PCA9685_BREAKOUT_ONLY_I2C, SamacSys_Parts:PCA9685_BREAKOUT_ONLY_I2C
- removed Y1: 32.768kHz, microbuilder:CRYSTALTHIN32K
- added C49: (no value), rcl:C-EUC0603
- added IC13: PCA9685PW, SamacSys_Parts:PCA9685PW
- added PROG: 3220-10-0300-00, SamacSys_Parts:3220-10-0300-00
- added R25: (no value), rcl:R-EU_R0603
- added SV1, SV2: (no value), con-lstb:MA10-1
- R7: value 47k -> 33R
Connections:
- removed net DISP_CS: IC12.PA12
- removed net DISP_DC: IC12.PA11
- removed net DISP_RS: IC12.PA26
- removed net GPS_PPS: IC12.PA14
- removed net ML_MON_CUR: IC12.PA19
- removed net ML_NFAULT: IC12.PB3
- removed net ML_PHASE: IC12.PA21
- removed net MOT_EN: IC12.PD8
- removed net MOT_MON_CUR: IC12.PA17
- removed net MOT_NFAULT: IC12.PB5
- removed net MOT_NSLEEP: IC12.PA28
- removed net MOT_PHASE: IC12.PD9
- removed net MR_MON_CUR: IC12.PA18
- removed net MR_NFAULT: IC12.PD0
- removed net MR_PHASE: IC12.PD31
- removed net PA09_UART_RXD_0: IC12.PA9
- removed net PA10_UART_TXD_0: IC12.PA10
- removed net PA20_PERIMETER_SENDER: IC12.PA20
- removed net PA21_USB_N: D2.I/O_2, IC12.HSDM, J1.D-
- removed net PA22_USB_P: D2.I/O_1, IC12.HSDP, J1.D+
- removed net PA7_XIN32: C20.1, IC12.PA7, Y1.1
- removed net PA8_XOUT32: C21.1, IC12.PA8, Y1.2
- removed net PB01_SPI_4_SCK: IC12.PD19
- removed net PB10_SPI_4_MOSI: IC12.PD21
- removed net PB11_SPI_4_MISO: IC12.PD20
- removed net PB6_SWDIO_TMS: IC12.PB6, R8.1, SWD.2
- removed net PB7_SWCLK_TCK: IC12.PB7, R9.1, SWD.4
- removed net PD25_UART_RXD_2: IC12.PD25
- removed net PD26_UART_TXD_2: IC12.PD26
- removed net SENSOR_SCL: IC12.PA4
- removed net SENSOR_SDA: IC12.PA3
- removed net SPI_1_CS: IC8.PC3
- removed net SPI_1_MISO: IC8.PC1
- removed net SPI_1_MOSI: IC8.PC0
- removed net SPI_1_SCK: IC8.PC2
- removed net TARGET_RESET: C38.1, IC12.NRST, R17.1, SWD.10
- removed net TOUCH_CS: IC12.PA27
- removed net TOUCH_IRQ: IC12.PD18
- removed net UART_1_RXD: IC8.PC5
- removed net UART_1_TXD: IC8.PC4
- removed net VCCINT: C33.1, C34.1, C35.1, C36.1, C39.1, C40.1, C41.1, C42.1, C43.1, C44.1, IC12.VDDCORE_1, IC12.VDDCORE_2, IC12.VDDCORE_3, IC12.VDDCORE_4, IC12.VDDOUT, IC12.VDDPLL, IC12.VDDUTMIC
- new net AIN_00: C16.1, IC8.PD0, R11.2
- new net AIN_01: C17.1, IC8.PD1, R12.2
- new net AIN_02: C18.1, IC8.PD2, R13.2
- new net AIN_03: C19.1, IC8.PD3, R14.2
- new net AIN_04: C47.1, IC8.PD4, R18.2
- new net AIN_05: C48.1, IC8.PD5, R19.2
- new net AIN_06: C49.1, IC8.PD6, R25.2
- new net CURR_ALERT_CHRG: IC6.ALERT, IC8.PB0
- new net CURR_ALERT_M1: IC1.ALERT, IC8.PC1
- new net CURR_ALERT_M2: IC2.ALERT, IC8.PC0
- new net CURR_ALERT_M3: IC8.PB5, IC9.ALERT
- new net CURR_ALERT_M4: IC10.ALERT, IC8.PB4
- new net CURR_ALERT_M5: IC11.ALERT, IC8.PB1
- new net CURR_ALERT_SYS: IC3.ALERT, IC8.PA7
- new net N$37: IC8.PA4
- new net N$38: IC13.LED5, SV1.7
- new net N$40: IC13.LED6, SV1.8
- new net N$41: IC13.LED7, SV1.9
- new net N$42: IC13.LED9, SV2.3
- new net N$43: IC13.LED10, SV2.4
- new net N$44: IC13.LED11, SV2.5
- new net N$45: IC13.LED12, SV2.6
- new net N$46: IC13.LED13, SV2.7
- new net N$47: IC13.LED14, SV2.8
- new net N$48: IC13.LED15, SV2.9
- new net PWM_PCA9685_OE: IC13.!OE, IC8.PC2
- new net UART_2_RXD: IC8.PF5
- new net UART_2_TXD: IC8.PF4
- net +3V3: now also IC13.VDD, PROG.4, SV1.1, SV2.1; no longer C25.1, C26.1, C27.1, C28.1, C29.1, C30.1, C31.1, C32.1, C45.1, C46.1, IC12.VDDIN, IC12.VDDIO_1, IC12.VDDIO_2, IC12.VDDIO_3, IC12.VDDIO_4, IC12.VDDPLLUSB, IC12.VDDUTMII, IC12.VREFP, R9.2, SWD.1, U$3.VCC.
- net +5V: no longer D1.K
- net /RESET: now also C38.1, R17.1, R7.1
- net ADC_REGEN_SENS: now also R25.1
- net GND: now also C49.2, IC13.VSS, PROG.2, PROG.9, SV1.10, SV2.10; no longer C20.2, C21.2, C25.2, C26.2, C27.2, C28.2, C29.2, C30.2, C31.2, C32.2, C33.2, C34.2, C35.2, C36.2, C37.2, C39.2, C40.2, C41.2, C42.2, C43.2, C44.2, C45.2, C46.2, D2.GND, IC12.GND_1, IC12.GND_2, IC12.GND_3, IC12.GND_4, IC12.GND_5, IC12.GND_6, IC12.VREFN, J1.GND, R7.1, SWD.3, SWD.5, SWD.9, U$3.GND.
- net I2C_1_SCL: now also IC13.SCL; no longer U$3.SCL.
- net I2C_1_SDA: now also IC13.SDA; no longer U$3.SDA.
- net N$13: now also PROG.3, R8.1; no longer C37.1, D1.A, D2.VCC, J1.VBUS
- net N$14: now also IC13.LED8, SV2.2; no longer C18.1, R13.2
- net N$16: now also PROG.6; no longer IC12.TST
- net N$19: now also IC13.LED0, SV1.2; no longer C17.1, R12.2
- net N$23: now also IC13.LED1, SV1.3; no longer C16.1, R11.2
- net N$30: now also IC13.LED2, SV1.4; no longer C48.1, R19.2
- net N$35: now also IC13.LED3, SV1.5; no longer C47.1, R18.2
- net N$36: now also IC13.LED4, SV1.6; no longer C19.1, R14.2
- net SPI_0_CS: now also IC8.PE3; no longer IC8.PA7
- net SPI_0_MISO: now also IC8.PE1; no longer IC8.PA5
- net SPI_0_MOSI: now also IC8.PE0; no longer IC8.PA4
- net SPI_0_SCK: now also IC8.PE2; no longer IC8.PA6
Other:
- moved on the sheet: C38, IC7, IC8, R17, R7, R8
