File: Hardware/KiCad/RoboticLawnMower/i2c_io_pwm.kicad_sch (KiCad schematic)
At the start: 6 parts, among them U4 PCA9685PW, U5 PCA9557PW

Commit message: layout update
Connections:
- net +3.3V: now also U4.28 (VDD)
- net GND: now also U4.14 (VSS)
- net PWM_CH_4: now reaches U4.10 (LED4)
- net PWM_CH_5: now reaches U4.11 (LED5)
- net PWM_CH_6: now reaches U4.12 (LED6)
- net PWM_CH_7: now reaches U4.13 (LED7)
- net PWM_CH_8: now reaches U4.15 (LED8)
- net PWM_CH_9: now reaches U4.16 (LED9)
- net PWM_CH_10: now reaches U4.17 (LED10)
- net PWM_CH_11: now reaches U4.18 (LED11)
- net PWM_CH_12: now reaches U4.19 (LED12)
- net PWM_CH_13: now reaches U4.20 (LED13)
- net PWM_CH_14: now reaches U4.21 (LED14)
- net PWM_CH_15: now reaches U4.22 (LED15)
- net SCL: now reaches U4.26 (SCL)
- net SDA: now reaches U4.27 (SDA)
- net PWM_CH_0: now reaches U4.6 (LED0)
- net PWM_CH_1: now reaches U4.7 (LED1)
- net PWM_CH_2: now reaches U4.8 (LED2)
- net PWM_CH_3: now reaches U4.9 (LED3)
Other:
- moved on the sheet: C12, C14

Commit message: schaltplan und layout
Parts:
- added R29, R31, R33: 10K, Resistor_SMD:R_0402_1005Metric, symbol Device:R
- added R30, R32, R34: N.P., Resistor_SMD:R_0402_1005Metric, symbol Device:R
Connections:
- net +3.3V: now also R29.1, R31.1, R33.1
- net GND: now also U4.24 (A5), U4.25 (EXTCLK), U4.4 (A3), U4.5 (A4), R30.2, R32.2, R34.2
- net at U4.1 (A0): now also R29.2, R30.1
- net at U4.2 (A1): now also R31.2, R32.1
- net ~{PCA_9685_OE}: now reaches U4.23 (~{OE})
- net at U4.3 (A2): now also R33.2, R34.1

Commit message: Layout
Parts:
- removed C11: 100n, Capacitor_SMD:C_0603_1608Metric, symbol Device:C
- removed C13: 1u, Capacitor_SMD:C_0603_1608Metric, symbol Device:C
- removed U5: PCA9557PW, Package_DFN_QFN:QFN-28-1EP_6x6mm_P0.65mm_EP4.25x4.25mm, symbol Interface_Expansion:MCP23017_ML
Changed lines of the file:
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@@
     (effects (font (size 1.27 1.27)) (justify right))
-  )
-  (symbol (lib_id "power:GND") (at 88.9 109.22 0) (unit 1)
-    (in_bom yes) (on_board yes) (fields_autoplaced)
-    (property "Reference" "#PWR02" (id 0) (at 88.9 115.57 0)
-      (effects (font (size 1.27 1.27)) hide)
-    )
-    (property "Value" "GND" (id 1) (at 88.9 114.3 0))
-    (property "Footprint" "" (id 2) (at 88.9 109.22 0)
-      (effects (font (size 1.27 1.27)) hide)
-    )
-    (property "Datasheet" "" (id 3) (at 88.9 109.22 0)
-      (effects (font (size 1.27 1.27)) hide)
-    )
-    (pin "1")
   )
   (symbol (lib_id "Device:R") (at 107.95 170.18 0) (unit 1)
@@
     (pin "1")
   )
-  (symbol (lib_id "Interface_Expansion:MCP23017_ML") (at 152.4 73.66 0) (unit 1)
-    (in_bom yes) (on_board yes)
-    (property "Reference" "U5" (id 0) (at 156.21 45.72 0)
-      (effects (font (size 1.27 1.27)) (justify left))
-    )
-    (property "Value" "PCA9557PW" (id 1) (at 156.21 48.26 0)
-      (effects (font (size 1.27 1.27)) (justify left))
-    )
-    (property "Footprint" "Package_DFN_QFN:QFN-28-1EP_6x6mm_P0.65mm_EP4.25x4.25mm" (id 2) (at 157.48 99.06 0)
-      (effects (font (size 1.27 1.27)) (justify left) hide)
-    )
-    (property "Datasheet" "http://ww1.microchip.com/downloads/en/DeviceDoc/20001952C.pdf" (id 3) (at 157.48 101.6 0)
-      (effects (font (size 1.27 1.27)) (justify left) hide)
-    )
-    (pin "1")
-    (pin "10")
-    (pin "11")
-    (pin "12")
-    (pin "13")
-    (pin "14")
-    (pin "15")
-    (pin "16")
-    (pin "17")
-    (pin "18")
-    (pin "19")
-    (pin "2")
-    (pin "20")
-    (pin "21")
-    (pin "22")
-    (pin "23")
-    (pin "24")
-    (pin "25")
-    (pin "26")
-    (pin "27")
-    (pin "28")
-    (pin "29")
-    (pin "3")
-    (pin "4")
-    (pin "5")
-    (pin "6")
-    (pin "7")
-    (pin "8")
-    (pin "9")
-  )
   (symbol (lib_id "power:GND") (at 107.95 204.47 0) (unit 1)
     (in_bom yes) (on_board yes) (fields_autoplaced)
@@
     (pin "2")
   )
-  (symbol (lib_id "power:+3.3V") (at 88.9 101.6 0) (unit 1)
-    (in_bom yes) (on_board yes) (fields_autoplaced)
-    (property "Reference" "#PWR01" (id 0) (at 88.9 105.41 0)
-      (effects (font (size 1.27 1.27)) hide)
-    )
-    (property "Value" "+3.3V" (id 1) (at 88.9 96.52 0))
-    (property "Footprint" "" (id 2) (at 88.9 101.6 0)
-      (effects (font (size 1.27 1.27)) hide)
-    )
-    (property "Datasheet" "" (id 3) (at 88.9 101.6 0)
-      (effects (font (size 1.27 1.27)) hide)
-    )
-    (pin "1")
-  )
   (symbol (lib_id "Device:R") (at 107.95 200.66 0) (unit 1)
     (in_bom yes) (on_board yes) (fields_autoplaced)
@@
     )
     (property "Datasheet" "~" (id 3) (at 107.95 200.66 0)
-      (effects (font (size 1.27 1.27)) hide)
-    )
-    (pin "1")
-    (pin "2")
-  )
-  (symbol (lib_id "Device:C") (at 100.33 105.41 0) (unit 1)
-    (in_bom yes) (on_board yes) (fields_autoplaced)
-    (property "Reference" "C13" (id 0) (at 104.14 104.1399 0)
-      (effects (font (size 1.27 1.27)) (justify left))
-    )
-    (property "Value" "1u" (id 1) (at 104.14 106.6799 0)
-      (effects (font (size 1.27 1.27)) (justify left))
-    )
-    (property "Footprint" "Capacitor_SMD:C_0603_1608Metric" (id 2) (at 101.2952 109.22 0)
-      (effects (font (size 1.27 1.27)) hide)
-    )
-    (property "Datasheet" "~" (id 3) (at 100.33 105.41 0)
       (effects (font (size 1.27 1.27)) hide)
     )
@@
     (pin "9")
   )
-  (symbol (lib_id "power:GND") (at 100.33 109.22 0) (unit 1)
-    (in_bom yes) (on_board yes) (fields_autoplaced)
-    (property "Reference" "#PWR06" (id 0) (at 100.33 115.57 0)
-      (effects (font (size 1.27 1.27)) hide)
-    )
-    (property "Value" "GND" (id 1) (at 100.33 114.3 0))
-    (property "Footprint" "" (id 2) (at 100.33 109.22 0)
-      (effects (font (size 1.27 1.27)) hide)
-    )
-    (property "Datasheet" "" (id 3) (at 100.33 109.22 0)
-      (effects (font (size 1.27 1.27)) hide)
-    )
-    (pin "1")
-  )
-  (symbol (lib_id "Device:C") (at 88.9 105.41 0) (unit 1)
-    (in_bom yes) (on_board yes) (fields_autoplaced)
-    (property "Reference" "C11" (id 0) (at 92.71 104.1399 0)
-      (effects (font (size 1.27 1.27)) (justify left))
-    )
-    (property "Value" "100n" (id 1) (at 92.71 106.6799 0)
-      (effects (font (size 1.27 1.27)) (justify left))
-    )
-    (property "Footprint" "Capacitor_SMD:C_0603_1608Metric" (id 2) (at 89.8652 109.22 0)
-      (effects (font (size 1.27 1.27)) hide)
-    )
-    (property "Datasheet" "~" (id 3) (at 88.9 105.41 0)
-      (effects (font (size 1.27 1.27)) hide)
-    )
-    (pin "1")
-    (pin "2")
-  )
   (symbol (lib_id "power:+3.3V") (at 107.95 148.59 0) (unit 1)
     (in_bom yes) (on_board yes) (fields_autoplaced)
@@
       (effects (font (size 1.27 1.27)) hide)
     )
-    (pin "1")
-  )
-  (symbol (lib_id "power:+3.3V") (at 100.33 101.6 0) (unit 1)
-    (in_bom yes) (on_board yes) (fields_autoplaced)
-    (property "Reference" "#PWR05" (id 0) (at 100.33 105.41 0)
-      (effects (font (size 1.27 1.27)) hide)
-    )
-    (property "Value" "+3.3V" (id 1) (at 100.33 96.52 0))
-    (property "Footprint" "" (id 2) (at 100.33 101.6 0)
-      (effects (font (size 1.27 1.27)) hide)
-    )
-    (property "Datasheet" "" (id 3) (at 100.33 101.6 0)
-      (effects (font (size 1.27 1.27)) hide)
-    )
