File: Hardware/KiCad/RoboticLawnMower/RoboticLawnMower.kicad_pcb (KiCad board)
At the start: 2 copper layers, 100.1 x 100 mm, 89 parts, among them J1 Conn_01x08, J10 Conn_01x02, J11 Conn_01x02, J2 Conn_01x08, J3 Conn_01x08, J4 Conn_01x08, J5 Conn_01x08, J6 Conn_01x04, J7 Conn_01x04, J8 Conn_01x04, J9 Conn_01x04, Q1 BSS123, Q10 Si7141DP, Q2 Si7141DP, Q3 BSS123, Q4 Si7141DP, Q5 BSS123, Q6 Si7141DP, Q7 BSS123, Q8 Si7141DP, Q9 BSS123, U1 INA233, U10 INA233, U11 INA233, U12 INA233, U13 INA233, U14 PCA9547BS, U2 AVR128DB48x-xPT, U3 ESP32-WROOM-32D, U4 PCA9685PW, U5 PCA9557PW, U6 LT1129-3.3_SOT223, U7 TSR_1-2450, U8 ADS1115IDGS, U9 ADS1115IDGS

Commit message: layout update
Parts:
- added C25: 5p6, Capacitor_SMD:C_0603_1608Metric, F.Cu at (176.5, 83.8)
- added J12: Conn_02x05_Row_Letter_Last, Connector_PinHeader_1.27mm:PinHeader_2x05_P1.27mm_Vertical_SMD, F.Cu at (174.6, 76.2)
- added J13: Conn_01x04, Connector_JST:JST_XA_B04B-XASK-1-A_1x04_P2.50mm_Vertical, F.Cu at (111.1, 47.6)
- added R26: 47K, Resistor_SMD:R_0603_1608Metric, F.Cu at (172.5, 83.8)
- added R27: 33R, Resistor_SMD:R_0603_1608Metric, F.Cu at (182.2, 77.9)
- added R28: 47K, Resistor_SMD:R_0603_1608Metric, F.Cu at (182.2, 75.4)
- added Y1: 32.768kHz, Crystal:Crystal_SMD_3215-2Pin_3.2x1.5mm, F.Cu at (135.3, 71.8)
- C3, C4, C5, C6, Q10, Q3, Q4, R10, R11, R22, R9, U10, U11, U13: moved to B.Cu
- moved R19 112.4 mm to (111.6, 114.5), turned to 180 degrees
- moved R18 105.9 mm to (113.7, 112.4)
- moved R10 84.5 mm to (159.4, 126.4)
- moved R9 80.0 mm to (159.4, 124.5), turned to 180 degrees
- moved R16 74.7 mm to (155.6, 88.9)
- moved R15 74.7 mm to (151.6, 88.9)
- moved R13 58.2 mm to (186.1, 97.2), turned to 180 degrees
- moved R12 53.9 mm to (186.1, 95.2)
- moved U4 35.6 mm to (139.1, 125.1), turned to 180 degrees
- moved U2 31.7 mm to (128.3, 78.7)
- moved R22 21.0 mm to (151.8, 141.0), turned to 180 degrees
- moved R17 20.9 mm to (156.8, 103.5)
- moved R24 20.9 mm to (160.9, 103.5)
- moved R23 20.7 mm to (184.8, 112.4)
- moved C3 17.6 mm to (146.1, 127.6), turned to 90 degrees
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Connections:
- J1 pad 6: /Motor_M1/MOT_Z/F (DIR) -> /PWM_CH_0
- J1 pad 7: /Motor_M1/MOT_VEL -> /PWM_CH_1
- J2 pad 6: /Motor_M2/MOT_Z/F (DIR) -> /PWM_CH_2
- J2 pad 7: /Motor_M2/MOT_VEL -> /PWM_CH_3
- J3 pad 6: /Motor_M3/MOT_Z/F (DIR) -> /PWM_CH_4
- J3 pad 7: /Motor_M3/MOT_VEL -> /PWM_CH_5
- J4 pad 6: /Motor_M4/MOT_Z/F (DIR) -> /PWM_CH_6
- J4 pad 7: /Motor_M4/MOT_VEL -> /PWM_CH_7
- J5 pad 6: /Motor_M5/MOT_Z/F (DIR) -> /PWM_CH_8
- J5 pad 7: /Motor_M5/MOT_VEL -> /PWM_CH_9
- R12 pad 1: /Motor_M3/POW_EN -> /Motor_M3/MOT_ENABLE
- R15 pad 1: /Motor_M4/POW_EN -> /Motor_M4/MOT_ENABLE
- R18 pad 1: /Motor_M5/POW_EN -> /Motor_M5/MOT_ENABLE
- R6 pad 1: /Motor_M1/POW_EN -> /Motor_M1/MOT_ENABLE
- R9 pad 1: /Motor_M2/POW_EN -> /Motor_M2/MOT_ENABLE
- U1 pad 4: /Motor_M1/SDA -> /I2C_1_SDA
- U1 pad 5: /Motor_M1/SCL -> /I2C_1_SCL
- U10 pad 4: /Motor_M2/SDA -> /I2C_1_SDA
- U10 pad 5: /Motor_M2/SCL -> /I2C_1_SCL
- U11 pad 4: /Motor_M3/SDA -> /I2C_1_SDA
- U11 pad 5: /Motor_M3/SCL -> /I2C_1_SCL
- U12 pad 4: /Motor_M4/SDA -> /I2C_1_SDA
- U12 pad 5: /Motor_M4/SCL -> /I2C_1_SCL
- U13 pad 4: /Motor_M5/SDA -> /I2C_1_SDA
- U13 pad 5: /Motor_M5/SCL -> /I2C_1_SCL
- U14 pad 19: /i2c_smb_mux/SCL -> /i2c_analog/SCL
- U14 pad 20: /i2c_smb_mux/SDA -> /i2c_analog/SDA
- U2 pad 1: unconnected-(U2-Pad1) -> /i2c_smb_mux/ADR_1
- U2 pad 10: unconnected-(U2-Pad10) -> /uC/CURR_ALERT_M2
- U2 pad 11: unconnected-(U2-Pad11) -> /uC/CURR_ALERT_M1
- U2 pad 12: unconnected-(U2-Pad12) -> /uC/PWM_PCA_9685_OE
- U2 pad 14: unconnected-(U2-Pad14) -> +3.3V
- U2 pad 15: Net-(U2-Pad15) -> GND
- U2 pad 2: unconnected-(U2-Pad2) -> /i2c_smb_mux/ADR_2
- U2 pad 28: unconnected-(U2-Pad28) -> +3.3V
- U2 pad 29: unconnected-(U2-Pad29) -> GND
- U2 pad 3: unconnected-(U2-Pad3) -> /uC/CURR_ALERT_SYS
- U2 pad 34: unconnected-(U2-Pad34) -> Net-(U2-Pad34)
- U2 pad 35: unconnected-(U2-Pad35) -> Net-(U2-Pad35)
- U2 pad 4: unconnected-(U2-Pad4) -> /uC/CURR_ALERT_CHRG
- U2 pad 40: unconnected-(U2-Pad40) -> /uC/~{AVR_RERSET}
- U2 pad 41: unconnected-(U2-Pad41) -> /uC/AVR_UPDI
- U2 pad 42: unconnected-(U2-Pad42) -> +3.3V
- U2 pad 43: Net-(U2-Pad15) -> GND
- U2 pad 44: unconnected-(U2-Pad44) -> /uC/UART_0_TXD
- U2 pad 45: unconnected-(U2-Pad45) -> /uC/UART_0_RXD
- U2 pad 46: unconnected-(U2-Pad46) -> /i2c_analog/SDA
- U2 pad 47: unconnected-(U2-Pad47) -> /i2c_analog/SCL
- U2 pad 48: unconnected-(U2-Pad48) -> /i2c_smb_mux/ADR_0
- U2 pad 5: unconnected-(U2-Pad5) -> /uC/CURR_ALERT_M5
- U2 pad 6: unconnected-(U2-Pad6) -> /uC/I2C_1_SDA
- U2 pad 7: unconnected-(U2-Pad7) -> /uC/I2C_1_SCL
- U2 pad 8: unconnected-(U2-Pad8) -> /uC/CURR_ALERT_M4
- U2 pad 9: unconnected-(U2-Pad9) -> /uC/CURR_ALERT_M3
- U4 pad 10: unconnected-(U4-Pad10) -> /PWM_CH_4
- U4 pad 11: unconnected-(U4-Pad11) -> /PWM_CH_5
- U4 pad 12: unconnected-(U4-Pad12) -> /PWM_CH_6
- U4 pad 13: unconnected-(U4-Pad13) -> /PWM_CH_7
- U4 pad 14: unconnected-(U4-Pad14) -> GND
- U4 pad 15: unconnected-(U4-Pad15) -> /PWM_CH_8
- U4 pad 16: unconnected-(U4-Pad16) -> /PWM_CH_9
- U4 pad 17: unconnected-(U4-Pad17) -> /PWM_CH_10
- U4 pad 18: unconnected-(U4-Pad18) -> /PWM_CH_11
- U4 pad 19: unconnected-(U4-Pad19) -> /PWM_CH_12
- U4 pad 20: unconnected-(U4-Pad20) -> /PWM_CH_13
- U4 pad 21: unconnected-(U4-Pad21) -> /PWM_CH_14
- U4 pad 22: unconnected-(U4-Pad22) -> /PWM_CH_15
- U4 pad 26: unconnected-(U4-Pad26) -> /I2C_1_SCL
- U4 pad 27: unconnected-(U4-Pad27) -> /I2C_1_SDA
- U4 pad 28: unconnected-(U4-Pad28) -> +3.3V
- U4 pad 6: unconnected-(U4-Pad6) -> /PWM_CH_0
- U4 pad 7: unconnected-(U4-Pad7) -> /PWM_CH_1
- U4 pad 8: unconnected-(U4-Pad8) -> /PWM_CH_2
- U4 pad 9: unconnected-(U4-Pad9) -> /PWM_CH_3
Routing:
- net /PWM_CH_9: track 0.00 -> 44.1 mm
- net /PWM_CH_0: track 0.00 -> 38.1 mm
- net /i2c_analog/SCL: track 0.00 -> 37.0 mm, vias 0 -> 1
- net /i2c_analog/SDA: track 0.00 -> 36.9 mm, vias 0 -> 1
- net /PWM_CH_8: track 0.00 -> 35.6 mm
- net /PWM_CH_1: track 0.00 -> 33.8 mm
- net /PWM_CH_4: track 0.00 -> 28.0 mm
- net /PWM_CH_5: track 0.00 -> 24.9 mm
- net /i2c_smb_mux/ADR_1: track 0.00 -> 22.7 mm, vias 0 -> 2
- net /i2c_smb_mux/ADR_0: track 0.00 -> 21.2 mm, vias 0 -> 2
- net /PWM_CH_3: track 0.00 -> 17.6 mm
- net /PWM_CH_7: track 0.00 -> 17.5 mm
- net +3.3V: track 7.06 -> 24.1 mm
- net /PWM_CH_6: track 0.00 -> 16.0 mm
- net /PWM_CH_2: track 0.00 -> 15.6 mm
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
Commit message: schaltplan und layout
Parts:
- removed Q10, Q6, Q8: Si7141DP, Package_SO:PowerPAK_SO-8_Single
- removed Q5, Q7, Q9: BSS123, Package_TO_SOT_SMD:SOT-23
- removed R19: 1M, Resistor_SMD:R_0603_1608Metric
- removed R20: 1K, Resistor_SMD:R_0603_1608Metric
- removed R21, R22, R23, R24, R25: 100k, Resistor_SMD:R_0603_1608Metric
- added D1: LED_GREEN, LED_SMD:LED_0603_1608Metric, F.Cu at (145.1, 129.5)
- added D2: LED_GREEN, LED_SMD:LED_0603_1608Metric, F.Cu at (145.1, 116.8)
- added D3: LED_GREEN, LED_SMD:LED_0603_1608Metric, F.Cu at (145.0, 104.1)
- added D4: LED_GREEN, LED_SMD:LED_0603_1608Metric, F.Cu at (145.0, 91.7)
- added D5: LED_GREEN, LED_SMD:LED_0603_1608Metric, F.Cu at (100.8, 129.8)
- added R29: 10K, Resistor_SMD:R_0402_1005Metric, F.Cu at (134.9, 121.2)
- added R30: N.P., Resistor_SMD:R_0402_1005Metric, F.Cu at (139.7, 117.6)
- added R31: 10K, Resistor_SMD:R_0402_1005Metric, F.Cu at (134.9, 122.4)
- added R32: N.P., Resistor_SMD:R_0402_1005Metric, F.Cu at (138.4, 117.6)
- added R33: 10K, Resistor_SMD:R_0402_1005Metric, F.Cu at (134.9, 123.7)
- added R34: N.P., Resistor_SMD:R_0402_1005Metric, F.Cu at (137.2, 117.6)
- C1, C2, C3, C4, C5, C6, Q4, U1, U10, U11, U13: moved to F.Cu
- Q2: value Si7141DP -> BSS123; footprint Package_SO:PowerPAK_SO-8_Single -> Package_TO_SOT_SMD:SOT-23
- Q3: value BSS123 -> Si7141DP; footprint Package_TO_SOT_SMD:SOT-23 -> Package_SO:PowerPAK_SO-8_Single; moved to F.Cu
- R10: value 1M -> 100k; moved to F.Cu
- R11: value 1K -> 100k; moved to F.Cu
- R12: value 100R -> 1K
- R13: value 1M -> 1K
- R14, R17: value 1K -> 2k2
- R15, R18: value 100R -> 2k2
- R16: value 1M -> 2k2
- R7: value 1M -> 100R
- R8: value 1K -> 1M
- R9: value 100R -> 1M; moved to F.Cu
- moved R12 95.3 mm to (118.5, 162.6), turned to 180 degrees
- moved Q1 73.0 mm to (122.4, 162.6), turned to 180 degrees
- moved R6 71.9 mm to (126.7, 162.6), turned to -90 degrees
- moved R8 70.1 mm to (125.2, 162.6), turned to 90 degrees
- moved H5 62.5 mm to (136.9, 139.2)
- moved R10 53.6 mm to (117.0, 159.3), turned to -90 degrees
- moved R14 49.1 mm to (145.1, 131.3), turned to 180 degrees
- moved R13 48.7 mm to (163.3, 140.2)
- moved C11 48.0 mm to (203.7, 57.2)
- moved C12 48.0 mm to (203.7, 59.7)
- moved C13 48.0 mm to (199.7, 59.7)
- moved C14 48.0 mm to (199.7, 57.2)
- moved C19 48.0 mm to (203.7, 49.2)
- moved C20 48.0 mm to (199.7, 49.2)
- moved C21 48.0 mm to (203.7, 46.7)
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Connections:
- C1 pad 2: GNDPWR -> GND
- C10 pad 2: GNDPWR -> GND
- C2 pad 2: GNDPWR -> GND
- C3 pad 2: GNDPWR -> GND
- C4 pad 2: GNDPWR -> GND
- C5 pad 2: GNDPWR -> GND
- C6 pad 2: GNDPWR -> GND
- C7 pad 2: GNDPWR -> GND
- C8 pad 2: GNDPWR -> GND
- C9 pad 2: GNDPWR -> GND
- J1 pad 2: GNDPWR -> GND
- J1 pad 4: /Motor_M1/MOT_ENABLE -> /Motor_M1..4_EN
- J1 pad 8: GNDPWR -> GND
- J10 pad 2: GNDPWR -> GND
- J11 pad 1: /Motor_M1/UBATT -> +BATT
- J11 pad 2: GNDPWR -> GND
- J2 pad 2: GNDPWR -> GND
- J2 pad 4: /Motor_M2/MOT_ENABLE -> /Motor_M1..4_EN
- J2 pad 8: GNDPWR -> GND
- J3 pad 2: GNDPWR -> GND
- J3 pad 4: /Motor_M3/MOT_ENABLE -> /Motor_M1..4_EN
- J3 pad 8: GNDPWR -> GND
- J4 pad 2: GNDPWR -> GND
- J4 pad 4: /Motor_M4/MOT_ENABLE -> /Motor_M1..4_EN
- J4 pad 8: GNDPWR -> GND
- J5 pad 2: GNDPWR -> GND
- J5 pad 4: /Motor_M5/MOT_ENABLE -> /Motor_M5_EN
- J5 pad 8: GNDPWR -> GND
- Q1 pad 2: GNDPWR -> GND
- Q2 pad 1: /Motor_M1/UBATT -> Net-(Q2-Pad1)
- Q2 pad 2: /Motor_M1/UBATT -> GND
- Q2 pad 3: /Motor_M1/UBATT -> Net-(Q2-Pad3)
- Q3 pad 1: Net-(Q3-Pad1) -> +BATT
- Q3 pad 2: GNDPWR -> +BATT
- Q3 pad 3: Net-(Q3-Pad3) -> +BATT
- Q4 pad 1: /Motor_M1/UBATT -> +BATT
- Q4 pad 2: /Motor_M1/UBATT -> +BATT
- Q4 pad 3: /Motor_M1/UBATT -> +BATT
- Q4 pad 5: Net-(Q4-Pad5) -> /Motor_M1/UBATT
- R1 pad 2: Net-(Q2-Pad5) -> /Motor_M1/UBATT
- R10 pad 1: Net-(Q3-Pad1) -> +BATT
- R10 pad 2: GNDPWR -> Net-(Q3-Pad4)
- R11 pad 1: Net-(Q3-Pad3) -> +BATT
- R12 pad 1: /Motor_M3/MOT_ENABLE -> Net-(Q1-Pad3)
- R12 pad 2: Net-(Q5-Pad1) -> Net-(Q3-Pad4)
- R13 pad 1: Net-(Q5-Pad1) -> Net-(Q2-Pad3)
- R13 pad 2: GNDPWR -> Net-(Q4-Pad4)
- R14 pad 1: Net-(Q5-Pad3) -> /Motor_M1/MOT_5V_OUT
- R15 pad 1: /Motor_M4/MOT_ENABLE -> /Motor_M2/MOT_5V_OUT
- R15 pad 2: Net-(Q7-Pad1) -> Net-(D2-Pad2)
- R16 pad 1: Net-(Q7-Pad1) -> /Motor_M3/MOT_5V_OUT
- R16 pad 2: GNDPWR -> Net-(D3-Pad2)
- R17 pad 1: Net-(Q7-Pad3) -> /Motor_M4/MOT_5V_OUT
- R18 pad 1: /Motor_M5/MOT_ENABLE -> /Motor_M5/MOT_5V_OUT
- R2 pad 2: Net-(Q4-Pad5) -> /Motor_M1/UBATT
- R3 pad 2: Net-(Q6-Pad5) -> /Motor_M1/UBATT
- R4 pad 2: Net-(Q8-Pad5) -> /Motor_M1/UBATT
- R5 pad 2: Net-(Q10-Pad5) -> /Motor_M5/UBATT
- R6 pad 1: /Motor_M1/MOT_ENABLE -> /Motor_M5_EN
- R7 pad 1: Net-(Q1-Pad1) -> /Motor_M1..4_EN
- R7 pad 2: GNDPWR -> Net-(Q2-Pad1)
- R8 pad 1: Net-(Q1-Pad3) -> Net-(Q1-Pad1)
- R8 pad 2: Net-(Q2-Pad4) -> GND
- R9 pad 1: /Motor_M2/MOT_ENABLE -> Net-(Q2-Pad1)
- R9 pad 2: Net-(Q3-Pad1) -> GND
- U1 pad 1: /Motor_M1/ADR_1 -> GND
- U1 pad 2: /Motor_M1/ADR_0 -> GND
- U1 pad 4: /I2C_1_SDA -> /Motor_M1/SDA
- U1 pad 5: /I2C_1_SCL -> /Motor_M1/SCL
- U1 pad 7: GNDPWR -> GND
- U1 pad 8: Net-(Q2-Pad5) -> Net-(R1-Pad4)
- U10 pad 1: /Motor_M2/ADR_1 -> GND
- U10 pad 2: /Motor_M2/ADR_0 -> +3.3V
- U10 pad 4: /I2C_1_SDA -> /Motor_M1/SDA
- U10 pad 5: /I2C_1_SCL -> /Motor_M1/SCL
- U10 pad 7: GNDPWR -> GND
- U10 pad 8: Net-(Q4-Pad5) -> Net-(R2-Pad4)
- U11 pad 1: /Motor_M3/ADR_1 -> GND
- U11 pad 2: /Motor_M3/ADR_0 -> /Motor_M1/SDA
- U11 pad 4: /I2C_1_SDA -> /Motor_M1/SDA
- U11 pad 5: /I2C_1_SCL -> /Motor_M1/SCL
- U11 pad 7: GNDPWR -> GND
- U11 pad 8: Net-(Q6-Pad5) -> Net-(R3-Pad4)
- U12 pad 1: /Motor_M4/ADR_1 -> GND
- U12 pad 2: /Motor_M4/ADR_0 -> /Motor_M1/SCL
- U12 pad 4: /I2C_1_SDA -> /Motor_M1/SDA
- U12 pad 5: /I2C_1_SCL -> /Motor_M1/SCL
- U12 pad 7: GNDPWR -> GND
- U12 pad 8: Net-(Q8-Pad5) -> Net-(R4-Pad4)
- U13 pad 1: /Motor_M5/ADR_1 -> +3.3V
- U13 pad 2: /Motor_M5/ADR_0 -> GND
- U13 pad 4: /I2C_1_SDA -> /Motor_M1/SDA
- U13 pad 5: /I2C_1_SCL -> /Motor_M1/SCL
- U13 pad 7: GNDPWR -> GND
- U13 pad 8: Net-(Q10-Pad5) -> Net-(R5-Pad4)
- U2 pad 12: /uC/PWM_PCA_9685_OE -> /i2c_io_pwm/~{PCA_9685_OE}
- U2 pad 13: unconnected-(U2-Pad13) -> /Motor_M1..4_EN
- U2 pad 16: unconnected-(U2-Pad16) -> /Motor_M5_EN
- U2 pad 6: /uC/I2C_1_SDA -> /Motor_M1/SDA
- U2 pad 7: /uC/I2C_1_SCL -> /Motor_M1/SCL
- U4 pad 1: unconnected-(U4-Pad1) -> Net-(U4-Pad1)
- U4 pad 2: unconnected-(U4-Pad2) -> Net-(U4-Pad2)
- U4 pad 23: unconnected-(U4-Pad23) -> /i2c_io_pwm/~{PCA_9685_OE}
- U4 pad 24: unconnected-(U4-Pad24) -> GND
- U4 pad 25: unconnected-(U4-Pad25) -> GND
- U4 pad 26: /I2C_1_SCL -> /Motor_M1/SCL
- U4 pad 27: /I2C_1_SDA -> /Motor_M1/SDA
- U4 pad 3: unconnected-(U4-Pad3) -> Net-(U4-Pad3)
- U4 pad 4: unconnected-(U4-Pad4) -> GND
- U4 pad 5: unconnected-(U4-Pad5) -> GND
- U7 pad 1: /Motor_M1/UBATT -> +BATT
Routing:
- net GND: track 2.04 -> 234.2 mm, vias 0 -> 3
- net /Motor_M1/SDA: track 0.00 -> 126.1 mm, vias 0 -> 2
- net /Motor_M1/SCL: track 0.00 -> 118.5 mm
- net +3.3V: track 24.1 -> 108.2 mm, vias 0 -> 8
- net /Motor_M1..4_EN: track 0.00 -> 63.7 mm, vias 0 -> 1
- net /Motor_M1/UBATT: track 113.0 -> 59.3 mm, vias 0 -> 4
- net /i2c_io_pwm/~{PCA_9685_OE}: track 0.00 -> 40.1 mm
- net /PWM_CH_6: track 16.0 -> 36.5 mm
- net /Motor_M5/MOT_5V_OUT: track 0.00 -> 19.1 mm
- net /Motor_M1/MOT_5V_OUT: track 0.00 -> 19.0 mm
- net /Motor_M2/MOT_5V_OUT: track 0.00 -> 18.6 mm
- net /Motor_M3/MOT_5V_OUT: track 0.00 -> 18.2 mm
- net /Motor_M4/MOT_5V_OUT: track 0.00 -> 17.9 mm
- net /PWM_CH_7: track 17.5 -> 33.5 mm
- net /PWM_CH_9: track 44.1 -> 31.6 mm
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
Commit message: layout
Parts:
- moved C17 100.7 mm to (113.0, 116.1)
- moved C18 96.4 mm to (113.0, 114.3)
- moved C15 95.3 mm to (112.5, 103.1)
- moved C16 92.1 mm to (112.6, 104.9)
- moved H5 33.8 mm to (137.7, 105.4)
- moved U7 23.8 mm to (106.3, 112.4), turned to 90 degrees
- moved R12 22.4 mm to (119.4, 140.2)
- moved R6 21.8 mm to (119.4, 142.0), turned to 0 degrees
- moved Q1 21.6 mm to (123.2, 141.0)
- moved Q3 21.6 mm to (122.8, 136.4)
- moved R10 21.6 mm to (117.9, 137.7)
- moved R8 21.6 mm to (126.0, 141.0)
- moved U6 17.2 mm to (115.1, 109.7)
- moved J11 9.40 mm to (94.0, 122.4)
- moved Y1 5.08 mm to (136.4, 76.7)
Routing:
- net GND: track 234.2 -> 379.7 mm, vias 3 -> 1
- net +BATT: track 4.52 -> 125.2 mm, vias 0 -> 2
- net /Motor_M1..4_EN: track 63.7 -> 161.5 mm, vias 1 -> 0
- net /Motor_M1/SDA: track 126.1 -> 196.2 mm, vias 2 -> 4
- net /Motor_M1/SCL: track 118.5 -> 186.7 mm
- net /Motor_M5_EN: track 0.00 -> 67.5 mm
- net /Motor_M5/MOT_SIGNAL: track 0.00 -> 41.1 mm
- net +3.3V: track 108.2 -> 122.0 mm, vias 8 -> 9
- net /Motor_M5/UBATT: track 0.00 -> 8.24 mm
- net Net-(Q1-Pad1): track 0.00 -> 5.86 mm
- net Net-(J5-Pad1): track 0.00 -> 5.68 mm
- net +5V: track 0.00 -> 5.62 mm
- net Net-(Q3-Pad4): track 0.00 -> 4.57 mm
- net Net-(Q1-Pad3): track 0.00 -> 2.76 mm
- net /Motor_M5/MOT_5V_OUT: track 19.1 -> 21.7 mm
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
Commit message: layout
Parts:
- moved C20 23.0 mm to (177.6, 55.6)
- moved C19 23.0 mm to (181.6, 55.6)
- moved C13 22.8 mm to (177.6, 65.5)
- moved C22 22.8 mm to (177.6, 52.6)
- moved C21 22.8 mm to (181.6, 52.6)
- moved C12 22.8 mm to (181.6, 65.5)
- moved C23 22.8 mm to (181.1, 69.8)
- moved C24 22.8 mm to (177.1, 69.8)
- moved C14 22.5 mm to (177.6, 61.7)
- moved C11 22.5 mm to (181.6, 61.7)
- moved U9 18.2 mm to (130.0, 58.7)
- moved U8 17.6 mm to (130.0, 53.6)
Routing:
- net +5V: track 5.62 -> 10.2 mm
- net +3.3V: track 122.0 -> 126.2 mm
- net /Motor_M1..4_EN: track 161.5 -> 163.8 mm, vias 0 -> 1
- net GND: track 379.7 -> 381.5 mm
- added copper zone on F.Cu, net GND

Commit message: Layout
Parts:
- added R19: 10K, Resistor_SMD:R_0603_1608Metric, B.Cu at (115.3, 58.7)
- added R20: 4k7, Resistor_SMD:R_0603_1608Metric, B.Cu at (106.2, 59.2)
- added R21: 4k7, Resistor_SMD:R_0603_1608Metric, B.Cu at (106.2, 56.6)
- added R22: 4k7, Resistor_SMD:R_0603_1608Metric, B.Cu at (96.3, 59.2)
- added R23: 4k7, Resistor_SMD:R_0603_1608Metric, B.Cu at (96.3, 56.6)
- added R24: 4k7, Resistor_SMD:R_0603_1608Metric, B.Cu at (96.0, 74.9)
- added R25: 4k7, Resistor_SMD:R_0603_1608Metric, B.Cu at (96.0, 72.4)
- added R35: 4k7, Resistor_SMD:R_0603_1608Metric, B.Cu at (106.2, 74.9)
- added R36: 4k7, Resistor_SMD:R_0603_1608Metric, B.Cu at (106.2, 72.4)
- added R37: 10K, Resistor_SMD:R_0402_1005Metric, B.Cu at (115.8, 65.3)
- added R38: N.P., Resistor_SMD:R_0402_1005Metric, B.Cu at (115.8, 62.5)
- added R39: 10K, Resistor_SMD:R_0402_1005Metric, B.Cu at (114.6, 65.3)
- added R40: N.P., Resistor_SMD:R_0402_1005Metric, B.Cu at (114.6, 62.5)
- added R41: 4k7, Resistor_SMD:R_0603_1608Metric, F.Cu at (118.6, 78.0)
- added R42: 4k7, Resistor_SMD:R_0603_1608Metric, F.Cu at (118.6, 79.5)
Connections:
- U14 pad 18: /i2c_smb_mux/ADR_2 -> GND
- U14 pad 22: /i2c_smb_mux/ADR_0 -> Net-(R37-Pad2)
- U14 pad 23: /i2c_smb_mux/ADR_1 -> Net-(R39-Pad2)
- U2 pad 1: /i2c_smb_mux/ADR_1 -> unconnected-(U2-Pad1)
- U2 pad 2: /i2c_smb_mux/ADR_2 -> unconnected-(U2-Pad2)
- U2 pad 48: /i2c_smb_mux/ADR_0 -> /i2c_smb_mux/~{RESET}
Routing:
- net +3.3V: track 126.2 -> 286.6 mm, vias 9 -> 11
- net /Motor_M1/MOT_SIGNAL: track 0.00 -> 57.2 mm
- net /Motor_M2/MOT_SIGNAL: track 0.00 -> 47.3 mm
- net /Motor_M3/MOT_SIGNAL: track 0.00 -> 37.2 mm
- net /i2c_smb_mux/~{RESET}: track 0.00 -> 26.2 mm, vias 0 -> 2
- net /Motor_M4/MOT_SIGNAL: track 0.00 -> 25.9 mm
- net /i2c_smb_mux/ADR_1: track 22.7 -> 0.00 mm, vias 2 -> 0
- net /i2c_smb_mux/ADR_0: track 21.2 -> 0.00 mm, vias 2 -> 0
- net /i2c_smb_mux/ADR_2: track 14.9 -> 0.00 mm
- net Net-(R39-Pad2): track 0.00 -> 12.3 mm, vias 0 -> 1
- net Net-(R37-Pad2): track 0.00 -> 9.04 mm, vias 0 -> 1
- net /Motor_M1/SDA: track 196.2 -> 201.3 mm
- net /Motor_M1/SCL: track 186.7 -> 191.6 mm
- net Net-(J7-Pad2): track 26.2 -> 28.7 mm
- net Net-(J7-Pad3): track 28.1 -> 30.6 mm
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
Commit message: Layout
Parts:
- removed C11: 100n, Capacitor_SMD:C_0603_1608Metric
- removed C13: 1u, Capacitor_SMD:C_0603_1608Metric
- removed U5: PCA9557PW, Package_DFN_QFN:QFN-28-1EP_6x6mm_P0.65mm_EP4.25x4.25mm
- added C26: 10n, Capacitor_SMD:C_0603_1608Metric, B.Cu at (136.4, 53.1)
- added C27: 10n, Capacitor_SMD:C_0603_1608Metric, B.Cu at (155.4, 53.1)
- added C28: 10n, Capacitor_SMD:C_0603_1608Metric, B.Cu at (133.1, 53.1)
- added C29: 10n, Capacitor_SMD:C_0603_1608Metric, B.Cu at (152.1, 53.1)
- added C30: 10n, Capacitor_SMD:C_0603_1608Metric, B.Cu at (130.0, 53.1)
- added C31: 10n, Capacitor_SMD:C_0603_1608Metric, B.Cu at (149.1, 53.1)
- added C32: 10n, Capacitor_SMD:C_0603_1608Metric, B.Cu at (126.7, 53.1)
- added C33: 10n, Capacitor_SMD:C_0603_1608Metric, B.Cu at (145.8, 53.1)
- added J14: Conn_01x06, Connector_JST:JST_XA_B06B-XASK-1-A_1x06_P2.50mm_Vertical, F.Cu at (125.3, 47.5)
- added J15: Conn_01x06, Connector_JST:JST_XA_B06B-XASK-1-A_1x06_P2.50mm_Vertical, F.Cu at (144.4, 47.5)
- added J16: Conn_01x04, Connector_JST:JST_XA_B04B-XASK-1-A_1x04_P2.50mm_Vertical, F.Cu at (160.5, 71.6)
- added J17: Conn_01x04, Connector_JST:JST_XA_B04B-XASK-1-A_1x04_P2.50mm_Vertical, F.Cu at (163.1, 47.5)
- added R43: 1k, Resistor_SMD:R_0603_1608Metric, B.Cu at (127.5, 50.8)
- added R44: 1k, Resistor_SMD:R_0603_1608Metric, B.Cu at (129.3, 50.8)
- added R45: 1k, Resistor_SMD:R_0603_1608Metric, B.Cu at (133.9, 50.8)
- added R46: 1k, Resistor_SMD:R_0603_1608Metric, B.Cu at (135.6, 50.8)
- added R47: 1k, Resistor_SMD:R_0603_1608Metric, B.Cu at (146.6, 50.8)
- added R48: 1k, Resistor_SMD:R_0603_1608Metric, B.Cu at (148.3, 50.8)
- added R49: 1k, Resistor_SMD:R_0603_1608Metric, B.Cu at (152.9, 50.8)
- added R50: 1k, Resistor_SMD:R_0603_1608Metric, B.Cu at (154.7, 50.8)
- C19, C20, C21, C22, U8, U9: moved to B.Cu
- moved C14 78.2 mm to (130.6, 124.2)
- moved C12 76.6 mm to (130.6, 122.7)
- moved C23 68.0 mm to (114.3, 57.4), turned to 180 degrees
- moved C24 63.8 mm to (114.3, 58.9), turned to 180 degrees
- moved R26 47.4 mm to (129.0, 65.0), turned to -90 degrees
- moved C19 44.5 mm to (137.2, 55.9), turned to 90 degrees
- moved R27 43.8 mm to (139.4, 68.1), turned to -90 degrees
- moved C21 43.1 mm to (138.7, 55.9), turned to 90 degrees
- moved R28 41.8 mm to (141.0, 68.1), turned to -90 degrees
- moved J12 41.5 mm to (134.1, 67.3)
- moved C25 39.2 mm to (139.4, 71.1), turned to -90 degrees
- moved C22 21.8 mm to (156.2, 56.6)
- moved C20 21.5 mm to (156.2, 58.2)
- moved U9 20.7 mm to (150.6, 56.6)
- moved U3 15.2 mm to (175.0, 64.8), turned to -90 degrees
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Connections:
- U2 pad 10: /uC/CURR_ALERT_M2 -> unconnected-(U2-Pad10)
- U2 pad 11: /uC/CURR_ALERT_M1 -> unconnected-(U2-Pad11)
- U2 pad 3: /uC/CURR_ALERT_SYS -> unconnected-(U2-Pad3)
- U2 pad 4: /uC/CURR_ALERT_CHRG -> unconnected-(U2-Pad4)
- U2 pad 44: /uC/UART_0_TXD -> /WLAN/UART_TxD_uC
- U2 pad 45: /uC/UART_0_RXD -> /WLAN/UART_RxD_uC
- U2 pad 5: /uC/CURR_ALERT_M5 -> unconnected-(U2-Pad5)
- U2 pad 8: /uC/CURR_ALERT_M4 -> unconnected-(U2-Pad8)
- U2 pad 9: /uC/CURR_ALERT_M3 -> unconnected-(U2-Pad9)
- U3 pad 1: Net-(U3-Pad1) -> GND
- U3 pad 13: unconnected-(U3-Pad13) -> /WLAN/RGB_LED_1
- U3 pad 15: Net-(U3-Pad1) -> GND
- U3 pad 16: unconnected-(U3-Pad16) -> /WLAN/RGB_LED_0
- U3 pad 2: unconnected-(U3-Pad2) -> +3.3V
- U3 pad 26: unconnected-(U3-Pad26) -> Net-(U3-Pad26)
- U3 pad 29: unconnected-(U3-Pad29) -> Net-(U3-Pad29)
- U3 pad 34: unconnected-(U3-Pad34) -> /WLAN/UART_TxD_uC
- U3 pad 35: unconnected-(U3-Pad35) -> /WLAN/UART_RxD_uC
- U3 pad 38: Net-(U3-Pad1) -> GND
- U3 pad 39: Net-(U3-Pad1) -> GND
- U8 pad 1: unconnected-(U8-Pad1) -> GND
- U8 pad 4: unconnected-(U8-Pad4) -> Net-(C32-Pad1)
- U8 pad 5: unconnected-(U8-Pad5) -> Net-(C30-Pad1)
- U8 pad 6: unconnected-(U8-Pad6) -> Net-(C28-Pad1)
- U8 pad 7: unconnected-(U8-Pad7) -> Net-(C26-Pad1)
- U9 pad 1: unconnected-(U9-Pad1) -> +3.3V
- U9 pad 4: unconnected-(U9-Pad4) -> Net-(C33-Pad1)
- U9 pad 5: unconnected-(U9-Pad5) -> Net-(C31-Pad1)
- U9 pad 6: unconnected-(U9-Pad6) -> Net-(C29-Pad1)
- U9 pad 7: unconnected-(U9-Pad7) -> Net-(C27-Pad1)
Routing:
- net +3.3V: track 286.6 -> 532.0 mm, vias 11 -> 13
- net GND: track 383.3 -> 492.0 mm, vias 1 -> 20
- net /WLAN/UART_TxD_uC: track 0.00 -> 65.1 mm, vias 0 -> 2
- net /WLAN/UART_RxD_uC: track 0.00 -> 62.9 mm, vias 0 -> 2
- net /i2c_analog/SDA: track 36.9 -> 72.2 mm
- net /i2c_analog/SCL: track 37.0 -> 72.0 mm
- net Net-(U3-Pad29): track 0.00 -> 17.1 mm
- net /uC/AVR_UPDI: track 0.00 -> 16.8 mm
- net /WLAN/RGB_LED_0: track 0.00 -> 15.4 mm
- net /uC/~{AVR_RERSET}: track 0.00 -> 14.9 mm
- net Net-(U3-Pad26): track 0.00 -> 13.5 mm
- net /Motor_M1..4_EN: track 163.8 -> 176.6 mm, vias 1 -> 2
- net /WLAN/RGB_LED_1: track 0.00 -> 8.58 mm
- net Net-(C33-Pad1): track 0.00 -> 5.83 mm
- net Net-(C27-Pad1): track 0.00 -> 5.83 mm
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- added copper zone on B.Cu, net GND
