File: Hardware/KiCad/RoboticLawnMower/RoboticLawnMower.kicad_pcb (KiCad board)
At the start: 2 copper layers, 100.1 x 100 mm, 126 parts, among them J1 Conn_01x08, J10 Conn_01x02, J11 Conn_01x02, J12 Conn_02x05_Row_Letter_Last, J13 Conn_01x04, J14 Conn_01x06, J15 Conn_01x06, J16 Conn_01x04, J17 Conn_01x04, J2 Conn_01x08, J3 Conn_01x08, J4 Conn_01x08, J5 Conn_01x08, J6 Conn_01x04, J7 Conn_01x04, J8 Conn_01x04, J9 Conn_01x04, Q1 BSS123, Q2 BSS123, Q3 Si7141DP, Q4 Si7141DP, U1 INA233, U10 INA233, U11 INA233, U12 INA233, U13 INA233, U14 PCA9547BS, U2 AVR128DB48x-xPT, U3 ESP32-WROOM-32D, U4 PCA9685PW, U6 LT1129-3.3_SOT223, U7 TSR_1-2450, U8 ADS1115IDGS, U9 ADS1115IDGS, Y1 32.768kHz

Commit message: LAYOUT
Parts:
- added C11: 5p6, Capacitor_SMD:C_0603_1608Metric, F.Cu at (160.3, 65.5)
- added J18: Conn_02x05_Row_Letter_Last, Connector_PinHeader_1.27mm:PinHeader_2x05_P1.27mm_Vertical_SMD, F.Cu at (153.9, 63.8)
- added R51: 47K, Resistor_SMD:R_0603_1608Metric, F.Cu at (148.6, 61.7)
- added R52: 33R, Resistor_SMD:R_0603_1608Metric, F.Cu at (160.3, 63.8)
- added R53: 47K, Resistor_SMD:R_0603_1608Metric, F.Cu at (160.3, 62.0)
- added R54: 4k7, Resistor_SMD:R_0603_1608Metric, F.Cu at (141.5, 73.3)
- added R55: 4k7, Resistor_SMD:R_0603_1608Metric, F.Cu at (141.5, 75.0)
- added R56: N.P., Resistor_SMD:R_0402_1005Metric, F.Cu at (123.4, 81.8)
- added R57: N.P., Resistor_SMD:R_0402_1005Metric, F.Cu at (125.5, 81.8)
- added R58: N.P., Resistor_SMD:R_0402_1005Metric, F.Cu at (124.5, 81.8)
- added R59: 10R, Resistor_SMD:R_0402_1005Metric, F.Cu at (141.0, 77.3)
- added R60: N.P., Resistor_SMD:R_0402_1005Metric, F.Cu at (119.1, 76.7)
- added R61: 10R, Resistor_SMD:R_0402_1005Metric, F.Cu at (146.0, 81.6)
- added R62: 10R, Resistor_SMD:R_0402_1005Metric, F.Cu at (148.1, 81.6)
- added R63: N.P., Resistor_SMD:R_0402_1005Metric, F.Cu at (120.1, 76.7)
- added R64: 10R, Resistor_SMD:R_0402_1005Metric, F.Cu at (142.3, 77.3)
- added R65: 10R, Resistor_SMD:R_0402_1005Metric, F.Cu at (147.0, 81.6)
- added U5: AVR128DB48x-xPT, Package_QFP:TQFP-48_7x7mm_P0.5mm, F.Cu at (149.8, 74.0)
- added Y2: 32.768kHz, Crystal:Crystal_SMD_3215-2Pin_3.2x1.5mm, F.Cu at (158.0, 71.2)
- moved J16 53.7 mm to (214.1, 74.4)
- moved C17 30.9 mm to (105.6, 86.1), turned to 180 degrees
- moved C18 27.4 mm to (105.6, 87.9), turned to 180 degrees
- moved U6 20.8 mm to (103.5, 92.5), turned to 180 degrees
- moved C16 10.1 mm to (106.0, 97.3), turned to 180 degrees
- moved C15 7.63 mm to (106.1, 99.1), turned to 180 degrees
- moved J10 7.16 mm to (93.9, 99.9)
- moved R26 5.95 mm to (124.5, 61.2)
- moved C25 5.95 mm to (134.9, 67.3)
- moved J12 5.95 mm to (129.5, 63.5)
- moved R27 5.95 mm to (134.9, 64.3)
- moved R28 5.95 mm to (136.4, 64.3)
- moved R41 4.89 mm to (119.4, 73.2)
- moved R42 4.89 mm to (119.4, 74.7)
- moved Y1 4.88 mm to (135.6, 71.9)
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Connections:
- J10 pad 1: unconnected-(J10-Pad1) -> +BATT
- R41 pad 1: /Motor_M1/SDA -> Net-(R41-Pad1)
- R42 pad 1: /Motor_M1/SCL -> Net-(R42-Pad1)
- U2 pad 12: /i2c_io_pwm/~{PCA_9685_OE} -> Net-(U2-Pad12)
- U2 pad 13: /Motor_M1..4_EN -> Net-(U2-Pad13)
- U2 pad 16: /Motor_M5_EN -> Net-(U2-Pad16)
- U2 pad 6: /Motor_M1/SDA -> Net-(R41-Pad1)
- U2 pad 7: /Motor_M1/SCL -> Net-(R42-Pad1)
Routing:
- net /Motor_M1/SDA: track 203.9 -> 95.1 mm, vias 4 -> 2
- net /Motor_M1/SCL: track 193.5 -> 85.7 mm
- net +3.3V: track 532.0 -> 426.1 mm
- net /WLAN/UART_TxD_uC: track 65.1 -> 4.84 mm, vias 2 -> 1
- net /WLAN/UART_RxD_uC: track 62.9 -> 4.95 mm, vias 2 -> 1
- net /Motor_M1..4_EN: track 176.6 -> 140.4 mm, vias 2 -> 1
- net /PWM_CH_8: track 37.6 -> 3.17 mm
- net /i2c_io_pwm/~{PCA_9685_OE}: track 40.1 -> 8.00 mm
- net +BATT: track 125.2 -> 154.3 mm
- net /PWM_CH_9: track 29.8 -> 2.26 mm
- net /Motor_M5_EN: track 72.6 -> 48.5 mm, vias 1 -> 0
- net /Motor_M4/MOT_SIGNAL: track 25.9 -> 5.82 mm
- net GND: track 492.0 -> 472.1 mm, vias 20 -> 21
- net /Motor_M3/MOT_SIGNAL: track 37.2 -> 18.2 mm
- net /i2c_analog/SDA: track 72.2 -> 53.2 mm
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- removed copper zone on B.Cu, net GND
- removed copper zone on F.Cu, net GND

Commit message: bild hinzugefügt.
Parts:
- removed J17: Conn_01x04, Connector_JST:JST_XA_B04B-XASK-1-A_1x04_P2.50mm_Vertical
- removed U3: ESP32-WROOM-32D, RF_Module:ESP32-WROOM-32
- J16: value Conn_01x04 -> Conn_01x06; footprint Connector_JST:JST_XA_B04B-XASK-1-A_1x04_P2.50mm_Vertical -> Connector_PinHeader_2.54mm:PinHeader_1x06_P2.54mm_Vertical
- moved J16 102.2 mm to (112.0, 70.5), turned to 0 degrees
- moved R63 0.51 mm to (120.7, 76.7)
- moved R60 0.38 mm to (119.5, 76.7)
Connections:
- J16 pad 2: Net-(J16-Pad2) -> /uC/UART_0_TXD
- J16 pad 3: Net-(J16-Pad3) -> /uC/UART_0_RXD
- J16 pad 4: GND -> /uC/UART_0_XCK
- U2 pad 1: unconnected-(U2-Pad1) -> /uC/UART_0_RXD
- U2 pad 2: unconnected-(U2-Pad2) -> /uC/UART_0_XCK
- U2 pad 3: unconnected-(U2-Pad3) -> /uC/UART_0_XDIR
- U2 pad 4: unconnected-(U2-Pad4) -> Net-(U2-Pad4)
- U2 pad 44: /WLAN/UART_TxD_uC -> unconnected-(U2-Pad44)
- U2 pad 45: /WLAN/UART_RxD_uC -> /i2c_smb_mux/~{RESET}
- U2 pad 48: /i2c_smb_mux/~{RESET} -> /uC/UART_0_TXD
- U2 pad 5: unconnected-(U2-Pad5) -> Net-(U2-Pad5)
- U5 pad 44: /uC/MOTOR_CTR_UART_0_TXD -> Net-(U2-Pad5)
- U5 pad 45: /uC/MOTOR_CTR_UART_0_RXD -> Net-(U2-Pad4)
- U5 pad 46: /uC/MOTOR_CTR_I2C_0_SDA -> unconnected-(U5-Pad46)
- U5 pad 47: /uC/MOTOR_CTR_I2C_0_SCL -> unconnected-(U5-Pad47)
Routing:
- net +3.3V: track 426.1 -> 543.3 mm, vias 13 -> 17
- net /Motor_M1/SDA: track 95.1 -> 211.5 mm, vias 2 -> 5
- net /Motor_M1/SCL: track 85.7 -> 197.4 mm, vias 0 -> 4
- net /Motor_M5/MOT_SIGNAL: track 22.6 -> 78.5 mm, vias 0 -> 2
- net /i2c_io_pwm/~{PCA_9685_OE}: track 8.00 -> 60.9 mm, vias 0 -> 3
- net /Motor_M5_EN: track 48.5 -> 100.5 mm, vias 0 -> 2
- net /Motor_M1..4_EN: track 140.4 -> 181.8 mm, vias 1 -> 2
- net /PWM_CH_9: track 2.26 -> 35.4 mm, vias 0 -> 1
- net Net-(U2-Pad5): track 0.00 -> 30.8 mm, vias 0 -> 2
- net Net-(U2-Pad4): track 0.00 -> 28.8 mm, vias 0 -> 2
- net /PWM_CH_8: track 3.17 -> 30.7 mm, vias 0 -> 1
- net /uC/UART_0_XDIR: track 0.00 -> 17.9 mm
- net /uC/~{AVR_RERSET_1}: track 0.00 -> 17.1 mm
- net /uC/UART_0_XCK: track 0.00 -> 16.0 mm
- net /Motor_M5/MOT_5V_OUT: track 4.28 -> 19.5 mm, vias 0 -> 1
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- added copper zone on B.Cu, net GND
- added copper zone on F.Cu, net GND
