File: Hardware/KiCad/RoboticLawnMower/uC.kicad_sch (KiCad schematic)
At the start: 1 part, among them U2 AVR128DB48x-xPT

Commit message: layout update
Parts:
- added C25: 5p6, Capacitor_SMD:C_0603_1608Metric, symbol Device:C
- added J12: Conn_02x05_Row_Letter_Last, symbol Connector_Generic:Conn_02x05_Odd_Even
- added R26, R28: 47K, Resistor_SMD:R_0603_1608Metric, symbol Device:R
- added R27: 33R, Resistor_SMD:R_0603_1608Metric, symbol Device:R
- added Y1: 32.768kHz, symbol Device:Crystal
Connections:
- net SMB_MUX_ADR_1: now reaches U2.1 (PA5)
- net CURR_ALERT_M2: now reaches U2.10 (PC0)
- net CURR_ALERT_M1: now reaches U2.11 (PC1)
- net PWM_PCA_9685_OE: now reaches U2.12 (PC2)
- net +3.3V: now reaches U2.14 (VDDIO2)
- net +3.3V: now also U2.28 (AVDD), U2.42 (VDD), J12.4 (Pin_4), R26.1, R28.1
- net GND: now reaches U2.15 (GND), U2.43 (GND)
- net GND: now also U2.29 (AGND), C25.2, J12.2 (Pin_2), J12.9 (Pin_9)
- net SMB_MUX_ADR_2: now reaches U2.2 (PA6)
- net CURR_ALERT_SYS: now reaches U2.3 (PA7)
- net at U2.34 (XTAL32K1/PF0): now also Y1.2
- net at U2.35 (XTAL32K2/PF1): now also Y1.1
- net CURR_ALERT_CHRG: now reaches U2.4 (PB0)
- net ~{AVR_RERSET}: now reaches U2.40 (~{RESET}/PF6)
- net ~{AVR_RERSET}: now also C25.1, R27.2, R28.2
- net AVR_UPDI: now reaches U2.41 (UPDI)
- net AVR_UPDI: now also J12.3 (Pin_3), R26.2
- net UART_0_TXD: now reaches U2.44 (XTALHF1/PA0)
- net UART_0_RXD: now reaches U2.45 (XTALHF2/PA1)
- net I2C_0_SDA: now reaches U2.46 (PA2)
- net I2C_0_SCL: now reaches U2.47 (PA3)
- net SMB_MUX_ADR_0: now reaches U2.48 (PA4)
- net CURR_ALERT_M5: now reaches U2.5 (PB1)
- net I2C_1_SDA: now reaches U2.6 (PB2)
- net I2C_1_SCL: now reaches U2.7 (PB3)
- net CURR_ALERT_M4: now reaches U2.8 (PB4)
- net CURR_ALERT_M3: now reaches U2.9 (PB5)
- new net: J12.6 (Pin_6), R27.1
Other:
- moved on the sheet: U2

Commit message: schaltplan und layout
Connections:
- net Motor_M1..4_EN: now reaches U2.13 (PC3)
- net Motor_M5_EN: now reaches U2.16 (PC4)
- net PWM_PCA_9685_OE renamed ~{PCA_9685_OE}
Changed lines of the file:
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@@
   (junction (at 198.12 80.01) (diameter 0) (color 0 0 0 0)
   )
-  (bus_entry (at 266.7 109.22) (size 2.54 2.54)
-    (stroke (width 0) (type default) (color 0 0 0 0))
-  )
-  (bus_entry (at 266.7 114.3) (size 2.54 2.54)
-    (stroke (width 0) (type default) (color 0 0 0 0))
-  )
-  (bus_entry (at 266.7 116.84) (size 2.54 2.54)
-    (stroke (width 0) (type default) (color 0 0 0 0))
-  )
-  (bus_entry (at 266.7 119.38) (size 2.54 2.54)
-    (stroke (width 0) (type default) (color 0 0 0 0))
-  )
-  (bus_entry (at 266.7 121.92) (size 2.54 2.54)
-    (stroke (width 0) (type default) (color 0 0 0 0))
-  )
-  (bus_entry (at 266.7 124.46) (size 2.54 2.54)
-    (stroke (width 0) (type default) (color 0 0 0 0))
-  )
-  (bus_entry (at 266.7 127) (size 2.54 2.54)
-    (stroke (width 0) (type default) (color 0 0 0 0))
-  )
-  (bus_entry (at 266.7 132.08) (size 2.54 2.54)
-    (stroke (width 0) (type default) (color 0 0 0 0))
-  )
-  (bus_entry (at 266.7 134.62) (size 2.54 2.54)
-    (stroke (width 0) (type default) (color 0 0 0 0))
-  )
-  (bus_entry (at 266.7 137.16) (size 2.54 2.54)
+  (bus_entry (at 283.21 114.3) (size 2.54 2.54)
+    (stroke (width 0) (type default) (color 0 0 0 0))
+  )
+  (bus_entry (at 283.21 116.84) (size 2.54 2.54)
+    (stroke (width 0) (type default) (color 0 0 0 0))
+  )
+  (bus_entry (at 283.21 109.22) (size 2.54 2.54)
+    (stroke (width 0) (type default) (color 0 0 0 0))
+  )
+  (bus_entry (at 283.21 132.08) (size 2.54 2.54)
+    (stroke (width 0) (type default) (color 0 0 0 0))
+  )
+  (bus_entry (at 283.21 134.62) (size 2.54 2.54)
+    (stroke (width 0) (type default) (color 0 0 0 0))
+  )
+  (bus_entry (at 283.21 127) (size 2.54 2.54)
+    (stroke (width 0) (type default) (color 0 0 0 0))
+  )
+  (bus_entry (at 283.21 124.46) (size 2.54 2.54)
     (stroke (width 0) (type default) (color 0 0 0 0))
   )
@@
     (stroke (width 0) (type default) (color 0 0 0 0))
   )
-  (bus (pts (xy 269.24 129.54) (xy 269.24 134.62))
+  (bus (pts (xy 285.75 129.54) (xy 285.75 134.62))
     (stroke (width 0) (type default) (color 0 0 0 0))
   )
@@
     (stroke (width 0) (type default) (color 0 0 0 0))
   )
-  (wire (pts (xy 220.98 114.3) (xy 266.7 114.3))
-    (stroke (width 0) (type default) (color 0 0 0 0))
-  )
-  (bus (pts (xy 269.24 116.84) (xy 269.24 119.38))
+  (wire (pts (xy 220.98 114.3) (xy 283.21 114.3))
+    (stroke (width 0) (type default) (color 0 0 0 0))
+  )
+  (bus (pts (xy 285.75 116.84) (xy 285.75 119.38))
     (stroke (width 0) (type default) (color 0 0 0 0))
   )
@@
     (stroke (width 0) (type default) (color 0 0 0 0))
   )
-  (wire (pts (xy 220.98 109.22) (xy 266.7 109.22))
+  (wire (pts (xy 220.98 142.24) (xy 266.7 142.24))
+    (stroke (width 0) (type default) (color 0 0 0 0))
+  )
+  (wire (pts (xy 220.98 139.7) (xy 266.7 139.7))
+    (stroke (width 0) (type default) (color 0 0 0 0))
+  )
+  (wire (pts (xy 220.98 109.22) (xy 283.21 109.22))
     (stroke (width 0) (type default) (color 0 0 0 0))
   )
@@
     (stroke (width 0) (type default) (color 0 0 0 0))
   )
-  (bus (pts (xy 269.24 121.92) (xy 269.24 124.46))
-    (stroke (width 0) (type default) (color 0 0 0 0))
-  )
   (wire (pts (xy 57.15 55.88) (xy 57.15 58.42))
     (stroke (width 0) (type default) (color 0 0 0 0))
@@
     (stroke (width 0) (type default) (color 0 0 0 0))
   )
-  (bus (pts (xy 269.24 134.62) (xy 269.24 137.16))
+  (bus (pts (xy 285.75 134.62) (xy 285.75 137.16))
     (stroke (width 0) (type default) (color 0 0 0 0))
   )
@@
     (stroke (width 0) (type default) (color 0 0 0 0))
   )
-  (bus (pts (xy 269.24 119.38) (xy 269.24 121.92))
-    (stroke (width 0) (type default) (color 0 0 0 0))
-  )
   (wire (pts (xy 76.2 96.52) (xy 77.47 96.52))
     (stroke (width 0) (type default) (color 0 0 0 0))
@@
     (stroke (width 0) (type default) (color 0 0 0 0))
   )
-  (wire (pts (xy 220.98 116.84) (xy 266.7 116.84))
+  (wire (pts (xy 220.98 116.84) (xy 283.21 116.84))
     (stroke (width 0) (type default) (color 0 0 0 0))
   )
@@
     (stroke (width 0) (type default) (color 0 0 0 0))
   )
-  (wire (pts (xy 220.98 132.08) (xy 266.7 132.08))
-    (stroke (width 0) (type default) (color 0 0 0 0))
-  )
-  (bus (pts (xy 269.24 124.46) (xy 269.24 127))
+  (wire (pts (xy 220.98 132.08) (xy 283.21 132.08))
+    (stroke (width 0) (type default) (color 0 0 0 0))
+  )
+  (bus (pts (xy 285.75 119.38) (xy 285.75 127))
     (stroke (width 0) (type default) (color 0 0 0 0))
   )
@@
     (stroke (width 0) (type default) (color 0 0 0 0))
   )
-  (wire (pts (xy 220.98 134.62) (xy 266.7 134.62))
+  (wire (pts (xy 220.98 134.62) (xy 283.21 134.62))
     (stroke (width 0) (type default) (color 0 0 0 0))
   )
@@
     (stroke (width 0) (type default) (color 0 0 0 0))
   )
-  (wire (pts (xy 220.98 124.46) (xy 266.7 124.46))
+  (wire (pts (xy 220.98 124.46) (xy 283.21 124.46))
     (stroke (width 0) (type default) (color 0 0 0 0))
   )
@@
     (stroke (width 0) (type default) (color 0 0 0 0))
   )
-  (bus (pts (xy 269.24 111.76) (xy 269.24 116.84))
+  (bus (pts (xy 285.75 111.76) (xy 285.75 116.84))
     (stroke (width 0) (type default) (color 0 0 0 0))
   )
@@
     (stroke (width 0) (type default) (color 0 0 0 0))
   )
-  (bus (pts (xy 269.24 137.16) (xy 269.24 139.7))
-    (stroke (width 0) (type default) (color 0 0 0 0))
-  )
-  (wire (pts (xy 220.98 127) (xy 266.7 127))
+  (bus (pts (xy 285.75 137.16) (xy 285.75 139.7))
+    (stroke (width 0) (type default) (color 0 0 0 0))
+  )
+  (wire (pts (xy 220.98 127) (xy 283.21 127))
     (stroke (width 0) (type default) (color 0 0 0 0))
   )
@@
     (stroke (width 0) (type default) (color 0 0 0 0))
   )
-  (bus (pts (xy 269.24 139.7) (xy 279.4 139.7))
+  (bus (pts (xy 285.75 139.7) (xy 295.91 139.7))
     (stroke (width 0) (type default) (color 0 0 0 0))
   )
@@
     (stroke (width 0) (type default) (color 0 0 0 0))
   )
-  (bus (pts (xy 269.24 127) (xy 269.24 129.54))
-    (stroke (width 0) (type default) (color 0 0 0 0))
-  )
-  (label "I2C_1_SCL" (at 241.3 121.92 0)
-    (effects (font (size 1.27 1.27)) (justify left bottom))
+  (bus (pts (xy 285.75 127) (xy 285.75 129.54))
+    (stroke (width 0) (type default) (color 0 0 0 0))
   )
   (label "CURR_ALERT_M3" (at 241.3 127 0)
     (effects (font (size 1.27 1.27)) (justify left bottom))
   )
-  (label "PWM_PCA_9685_OE" (at 241.3 137.16 0)
-    (effects (font (size 1.27 1.27)) (justify left bottom))
-  )
-  (label "I2C_1_SDA" (at 241.3 119.38 0)
-    (effects (font (size 1.27 1.27)) (justify left bottom))
-  )
   (label "CURR_ALERT_M5" (at 241.3 116.84 0)
     (effects (font (size 1.27 1.27)) (justify left bottom))
@@
     (effects (font (size 1.27 1.27)) (justify left bottom))
   )
+  (hierarchical_label "I2C_1_SDA" (shape bidirectional) (at 266.7 119.38 0)
+    (effects (font (size 1.27 1.27)) (justify left))
+  )
   (hierarchical_label "I2C_0_SDA" (shape bidirectional) (at 266.7 96.52 0)
     (effects (font (size 1.27 1.27)) (justify left))
@@
     (effects (font (size 1.27 1.27)) (justify left))
   )
+  (hierarchical_label "I2C_1_SCL" (shape bidirectional) (at 266.7 121.92 0)
+    (effects (font (size 1.27 1.27)) (justify left))
+  )
   (hierarchical_label "I2C_0_SCL" (shape bidirectional) (at 266.7 99.06 0)
     (effects (font (size 1.27 1.27)) (justify left))
   )
+  (hierarchical_label "~{PCA_9685_OE}" (shape bidirectional) (at 266.7 137.16 0)
+    (effects (font (size 1.27 1.27)) (justify left))
+  )
   (hierarchical_label "SMB_MUX_ADR_0" (shape bidirectional) (at 266.7 101.6 0)
     (effects (font (size 1.27 1.27)) (justify left))
@@
     (effects (font (size 1.27 1.27)) (justify left))
   )
-  (hierarchical_label "MOTOR_CONTROL" (shape bidirectional) (at 279.4 139.7 0)
+  (hierarchical_label "MOTOR_CONTROL" (shape bidirectional) (at 295.91 139.7 0)
     (effects (font (size 1.27 1.27)) (justify left))
   )
@@
     (effects (font (size 1.27 1.27)) (justify left))
   )
+  (hierarchical_label "Motor_M1..4_EN" (shape bidirectional) (at 266.7 139.7 0)
+    (effects (font (size 1.27 1.27)) (justify left))
+  )
   (hierarchical_label "SMB_MUX_ADR_1" (shape bidirectional) (at 266.7 104.14 0)
     (effects (font (size 1.27 1.27)) (justify left))
   )
+  (hierarchical_label "Motor_M5_EN" (shape bidirectional) (at 266.7 142.24 0)
+    (effects (font (size 1.27 1.27)) (justify left))
+  )

Commit message: layout
Parts:
- J12: footprint (none) -> Connector_PinHeader_1.27mm:PinHeader_2x05_P1.27mm_Vertical_SMD
- Y1: footprint (none) -> Crystal:Crystal_SMD_3215-2Pin_3.2x1.5mm
Changed lines of the file:
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@@
     (property "Reference" "Y1" (id 0) (at 81.28 88.9 0))
     (property "Value" "32.768kHz" (id 1) (at 81.28 91.44 0))
-    (property "Footprint" "" (id 2) (at 81.28 96.52 0)
+    (property "Footprint" "Crystal:Crystal_SMD_3215-2Pin_3.2x1.5mm" (id 2) (at 81.28 96.52 0)
       (effects (font (size 1.27 1.27)) hide)
     )
@@
     (property "Reference" "J12" (id 0) (at 76.2 49.53 0))
     (property "Value" "Conn_02x05_Row_Letter_Last" (id 1) (at 76.2 52.07 0))
-    (property "Footprint" "" (id 2) (at 74.93 60.96 0)
+    (property "Footprint" "Connector_PinHeader_1.27mm:PinHeader_2x05_P1.27mm_Vertical_SMD" (id 2) (at 74.93 60.96 0)
       (effects (font (size 1.27 1.27)) hide)
     )

Commit message: Layout
Parts:
- added R41, R42: 4k7, Resistor_SMD:R_0603_1608Metric, symbol Device:R
Connections:
- net +3.3V: now also R41.2, R42.2
- net I2C_1_SCL: now also R42.1
- net I2C_1_SDA: now also R41.1
- net SMB_MUX_ADR_0 renamed ~{SMB_MUX_RESET}
- net SMB_MUX_ADR_1: no longer names the net of U2.1 (PA5)
- net SMB_MUX_ADR_2: no longer names the net of U2.2 (PA6)
Changed lines of the file:
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@@
 (kicad_sch (version 20211123) (generator eeschema)
   (paper "A3")
+  (junction (at 233.68 72.39) (diameter 0) (color 0 0 0 0)
+  )
   (junction (at 110.49 60.96) (diameter 0) (color 0 0 0 0)
   )
   (junction (at 57.15 58.42) (diameter 0) (color 0 0 0 0)
   )
+  (junction (at 236.22 121.92) (diameter 0) (color 0 0 0 0)
+  )
   (junction (at 198.12 163.83) (diameter 0) (color 0 0 0 0)
   )
@@
   (junction (at 198.12 80.01) (diameter 0) (color 0 0 0 0)
   )
+  (junction (at 233.68 119.38) (diameter 0) (color 0 0 0 0)
+  )
   (bus_entry (at 283.21 114.3) (size 2.54 2.54)
     (stroke (width 0) (type default) (color 0 0 0 0))
@@
     (stroke (width 0) (type default) (color 0 0 0 0))
   )
+  (wire (pts (xy 233.68 71.12) (xy 233.68 72.39))
+    (stroke (width 0) (type default) (color 0 0 0 0))
+  )
   (bus (pts (xy 285.75 129.54) (xy 285.75 134.62))
     (stroke (width 0) (type default) (color 0 0 0 0))
   )
+  (wire (pts (xy 220.98 101.6) (xy 266.7 101.6))
+    (stroke (width 0) (type default) (color 0 0 0 0))
+  )
   (wire (pts (xy 76.2 102.87) (xy 76.2 96.52))
     (stroke (width 0) (type default) (color 0 0 0 0))
   )
+  (wire (pts (xy 236.22 72.39) (xy 233.68 72.39))
+    (stroke (width 0) (type default) (color 0 0 0 0))
+  )
   (wire (pts (xy 220.98 114.3) (xy 283.21 114.3))
     (stroke (width 0) (type default) (color 0 0 0 0))
@@
     (stroke (width 0) (type default) (color 0 0 0 0))
   )
+  (wire (pts (xy 233.68 119.38) (xy 266.7 119.38))
+    (stroke (width 0) (type default) (color 0 0 0 0))
+  )
   (wire (pts (xy 200.66 80.01) (xy 200.66 83.82))
     (stroke (width 0) (type default) (color 0 0 0 0))
   )
+  (wire (pts (xy 236.22 121.92) (xy 266.7 121.92))
+    (stroke (width 0) (type default) (color 0 0 0 0))
+  )
   (wire (pts (xy 85.09 96.52) (xy 180.34 96.52))
     (stroke (width 0) (type default) (color 0 0 0 0))
@@
     (stroke (width 0) (type default) (color 0 0 0 0))
   )
+  (wire (pts (xy 233.68 82.55) (xy 233.68 119.38))
+    (stroke (width 0) (type default) (color 0 0 0 0))
+  )
   (wire (pts (xy 57.15 55.88) (xy 57.15 58.42))
     (stroke (width 0) (type default) (color 0 0 0 0))
@@
     (stroke (width 0) (type default) (color 0 0 0 0))
   )
-  (wire (pts (xy 220.98 104.14) (xy 266.7 104.14))
-    (stroke (width 0) (type default) (color 0 0 0 0))
-  )
-  (wire (pts (xy 220.98 101.6) (xy 266.7 101.6))
-    (stroke (width 0) (type default) (color 0 0 0 0))
-  )
   (wire (pts (xy 87.63 102.87) (xy 76.2 102.87))
     (stroke (width 0) (type default) (color 0 0 0 0))
@@
     (stroke (width 0) (type default) (color 0 0 0 0))
   )
+  (wire (pts (xy 236.22 74.93) (xy 236.22 72.39))
+    (stroke (width 0) (type default) (color 0 0 0 0))
+  )
   (wire (pts (xy 87.63 99.06) (xy 87.63 102.87))
     (stroke (width 0) (type default) (color 0 0 0 0))
@@
     (stroke (width 0) (type default) (color 0 0 0 0))
   )
+  (wire (pts (xy 233.68 72.39) (xy 233.68 74.93))
+    (stroke (width 0) (type default) (color 0 0 0 0))
+  )
   (wire (pts (xy 220.98 99.06) (xy 266.7 99.06))
     (stroke (width 0) (type default) (color 0 0 0 0))
@@
     (stroke (width 0) (type default) (color 0 0 0 0))
   )
+  (wire (pts (xy 236.22 82.55) (xy 236.22 121.92))
+    (stroke (width 0) (type default) (color 0 0 0 0))
+  )
   (wire (pts (xy 110.49 55.88) (xy 110.49 60.96))
     (stroke (width 0) (type default) (color 0 0 0 0))
@@
     (stroke (width 0) (type default) (color 0 0 0 0))
   )
-  (wire (pts (xy 220.98 119.38) (xy 266.7 119.38))
+  (wire (pts (xy 220.98 119.38) (xy 233.68 119.38))
     (stroke (width 0) (type default) (color 0 0 0 0))
   )
@@
     (stroke (width 0) (type default) (color 0 0 0 0))
   )
-  (wire (pts (xy 220.98 121.92) (xy 266.7 121.92))
+  (wire (pts (xy 220.98 121.92) (xy 236.22 121.92))
     (stroke (width 0) (type default) (color 0 0 0 0))
   )
@@
     (stroke (width 0) (type default) (color 0 0 0 0))
   )
-  (wire (pts (xy 220.98 106.68) (xy 266.7 106.68))
-    (stroke (width 0) (type default) (color 0 0 0 0))
-  )
   (wire (pts (xy 110.49 60.96) (xy 139.7 60.96))
     (stroke (width 0) (type default) (color 0 0 0 0))
@@
     (effects (font (size 1.27 1.27)) (justify left))
   )
-  (hierarchical_label "SMB_MUX_ADR_0" (shape bidirectional) (at 266.7 101.6 0)
-    (effects (font (size 1.27 1.27)) (justify left))
-  )
-  (hierarchical_label "SMB_MUX_ADR_2" (shape bidirectional) (at 266.7 106.68 0)
-    (effects (font (size 1.27 1.27)) (justify left))
-  )
   (hierarchical_label "MOTOR_CONTROL" (shape bidirectional) (at 295.91 139.7 0)
     (effects (font (size 1.27 1.27)) (justify left))
@@
     (effects (font (size 1.27 1.27)) (justify left))
   )
-  (hierarchical_label "SMB_MUX_ADR_1" (shape bidirectional) (at 266.7 104.14 0)
+  (hierarchical_label "~{SMB_MUX_RESET}" (shape output) (at 266.7 101.6 0)
     (effects (font (size 1.27 1.27)) (justify left))
   )
   (hierarchical_label "Motor_M5_EN" (shape bidirectional) (at 266.7 142.24 0)
     (effects (font (size 1.27 1.27)) (justify left))
+  )
+  (symbol (lib_id "Device:R") (at 236.22 78.74 180) (unit 1)
+    (in_bom yes) (on_board yes)
+    (property "Reference" "R42" (id 0) (at 238.76 82.55 90))
+    (property "Value" "4k7" (id 1) (at 236.22 78.74 90))
+    (property "Footprint" "Resistor_SMD:R_0603_1608Metric" (id 2) (at 237.998 78.74 90)
+      (effects (font (size 1.27 1.27)) hide)
+    )
+    (property "Datasheet" "~" (id 3) (at 236.22 78.74 0)
+      (effects (font (size 1.27 1.27)) hide)
+    )
+    (pin "1")
+    (pin "2")
   )
   (symbol (lib_id "Device:Crystal") (at 81.28 96.52 0) (unit 1)
@@
     )
     (property "Datasheet" "~" (id 3) (at 81.28 96.52 0)
+      (effects (font (size 1.27 1.27)) hide)
+    )
+    (pin "1")
+    (pin "2")
+  )
+  (symbol (lib_id "Device:R") (at 233.68 78.74 180) (unit 1)
+    (in_bom yes) (on_board yes)
+    (property "Reference" "R41" (id 0) (at 231.14 81.28 90))
+    (property "Value" "4k7" (id 1) (at 233.68 78.74 90))
+    (property "Footprint" "Resistor_SMD:R_0603_1608Metric" (id 2) (at 235.458 78.74 90)
+      (effects (font (size 1.27 1.27)) hide)
+    )
+    (property "Datasheet" "~" (id 3) (at 233.68 78.74 0)
       (effects (font (size 1.27 1.27)) hide)
     )
@@
       (effects (font (size 1.27 1.27)) hide)
     )
+    (pin "1")
+  )
+  (symbol (lib_id "power:+3.3V") (at 233.68 71.12 0) (unit 1)
+    (in_bom yes) (on_board yes) (fields_autoplaced)
+    (property "Reference" "#PWR070" (id 0) (at 233.68 74.93 0)
+      (effects (font (size 1.27 1.27)) hide)
+    )
+    (property "Value" "+3.3V" (id 1) (at 233.68 66.04 0))
+    (property "Footprint" "" (id 2) (at 233.68 71.12 0)
+      (effects (font (size 1.27 1.27)) hide)
+    )
+    (property "Datasheet" "" (id 3) (at 233.68 71.12 0)
+      (effects (font (size 1.27 1.27)) hide)
+    )
