File: Hardware/KiCad/RoboticLawnMower/RoboticLawnMower.kicad_sch (KiCad schematic)
At the start: 19 parts, among them J10 Conn_01x02, J11 Conn_01x02, Q1 BSS123, Q2 BSS123, Q3 Si7141DP, Q4 Si7141DP

Commit message: Schaltplan & Layout Änderung
Other:
- added sheet GPS (gps.kicad_sch)
- sheet Sensor ports: added Collision_Sensor_00, Collision_Sensor_01, Collision_Sensor_02; removed none
- sheet uC ports: added Collision_Sensor_00, Collision_Sensor_01, Collision_Sensor_02, GPS_PPS, GPS_RESET_EN, GPS_UART_3_RXD, GPS_UART_3_TXD; removed ~{SMB_MUX_RESET}

Commit message: Layout ready add gerber file
Parts:
- removed J10: Conn_01x02, Connector_Phoenix_MC:PhoenixContact_MCV_1,5_2-GF-3.81_1x02_P3.81mm_Vertical_ThreadedFlange_MountHole, symbol Connector_Generic:Conn_01x02
- added H6: MountingHole, MountingHole:MountingHole_3.2mm_M3, symbol Mechanical:MountingHole
Other:
- removed sheet charge
- sheet GPS ports: added GPS_MOD_EN; removed none
- sheet WLAN ports: added WLAN_MOD_EN; removed none
- sheet uC ports: added GPS_MOD_EN, WLAN_MOD_EN; removed none
- moved on the sheet: H1, H2, H3, H4, H5
