File: Hardware/KiCad/RoboticLawnMower/RoboticLawnMower.kicad_sch (KiCad schematic)
At the start: 19 parts, among them J11 Conn_01x02, Q1 BSS123, Q2 BSS123, Q3 Si7141DP, Q4 Si7141DP

Commit message: Redesign: - Controller - I2C pinning geändert - uvm
Other:
- added sheet RS485 (RS485.kicad_sch)
- sheet Motor_M1 ports: added RS485_A, RS485_B; removed none
- sheet Motor_M2 ports: added RS485_A, RS485_B; removed none
- sheet Motor_M3 ports: added RS485_A, RS485_B; removed none
- sheet Motor_M4 ports: added RS485_A, RS485_B; removed none
- sheet Motor_M5 ports: added RS485_A, RS485_B; removed none
- sheet i2c_analog ports: added I2C_2_SCL, I2C_2_SDA; removed SCL, SDA
- sheet i2c_smb_mux ports: added I2C_2_SCL, I2C_2_SDA; removed SCL, SDA
- sheet uC ports: added GPS_UART_RXD, GPS_UART_TXD, I2C_2_SCL, I2C_2_SDA, RS485_DIR, RS485_RX, RS485_TX, UART_RXD, UART_TXD, UART_XCK, UART_XDIR; removed GPS_UART_3_RXD, GPS_UART_3_TXD, I2C_0_SCL, I2C_0_SDA, UART_0_RXD, UART_0_TXD, UART_0_XCK, UART_0_XDIR
- note added: "I2C Adress PCA9685 0X47 PWM (ADDR = A0) ADS1115 0x48 ANALOG (ADDR = GND) ADS1115 0x49 ANALOG (ADDR = VCC) BMI180 0x69 ACC/GYR (SDO = VCC) 0x68 (SDO = GND) BME280 0x77 ENV (SDO = VCC) 0x76 (SDO = GND) LSM303 0x3A ACC 0x3C MAG INA228 0x40 M1 (A0 = GND | A1 = GND) INA228 0x41 M2 (A0 = VCC | A1 = GND) INA228 0x42 M3 (A0 = SDA | A1 = GND) INA228 0x43 M4 (A0 = SCL | A1 = GND) INA228 0x44 M5 (A0 = VCC |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"
- note added: "PWM CHANNEL: [PCA9685] CH0: M1 DIR CH1: M1 VEL CH2: M2 DIR CH3: M2 VEL CH4: M3 DIR CH5: M3 VEL CH6: M4 DIR CH7: M4 VEL CH8: LIGHT FRONT CH9: LIGHT BACK CH10: LIGHT FLASH CH11: CH12: CH13: CH14: M5 VEL CH15: M5 DIR"
- moved on the sheet: H1, H2, H3, H4, H5, H6

Commit message: change µC to STM32H573
Other:
- sheet uC ports: added MOT_SIG_5; removed none
Changed lines of the file:
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@@
 	(wire
 		(pts
+			(xy 302.26 232.41) (xy 330.2 232.41)
+		)
+		(stroke
+			(width 0)
+			(type default)
+		)
+	)
+	(wire
+		(pts
 			(xy 368.3 223.52) (xy 386.08 223.52)
 		)
@@
 	(wire
 		(pts
+			(xy 182.88 96.52) (xy 200.66 96.52)
+		)
+		(stroke
+			(width 0)
+			(type default)
+		)
+	)
+	(wire
+		(pts
 			(xy 132.08 44.45) (xy 132.08 27.94)
 		)
@@
 		)
 	)
+	(label "MOT_SIG_5"
+		(at 303.53 232.41 0)
+		(fields_autoplaced yes)
+		(effects
+			(font
+				(size 1.27 1.27)
+			)
+			(justify left bottom)
+		)
+	)
 	(label "PWM_CH_[0..15]"
 		(at 237.49 152.4 0)
@@
 		)
 	)
+	(label "MOT_SIG_5"
+		(at 191.77 96.52 0)
+		(fields_autoplaced yes)
+		(effects
+			(font
+				(size 1.27 1.27)
+			)
+			(justify left bottom)
+		)
+	)
 	(label "Motor_M5_EN"
 		(at 298.45 229.87 0)
@@
 			(effects
 				(font
+					(size 1.27 1.27)
+				)
+				(justify right)
+			)
+		)
+		(pin "MOT_SIG_5" input
+			(at 182.88 96.52 0)
+			(effects
+				(font
