File: Hardware/KiCad/RoboticLawnMower/wlan.kicad_sch (KiCad schematic)
At the start: 1 part, among them U3 mini_esp32

Commit message: Layout ready add gerber file
Parts:
- added Q5: Si7141DP, Package_SO:PowerPAK_SO-8_Single, symbol Transistor_FET:Si7141DP
- added Q6: BSS123, Package_TO_SOT_SMD:SOT-23, symbol Transistor_FET:BSS123
- added R22: 1K, Resistor_SMD:R_0603_1608Metric, symbol Device:R
- added R23: 100k, Resistor_SMD:R_0603_1608Metric, symbol Device:R
- added R24: 1M, Resistor_SMD:R_0603_1608Metric, symbol Device:R
- added R25: 100R, Resistor_SMD:R_0603_1608Metric, symbol Device:R
Connections:
- net +3.3V: now also Q5.1 (S), Q5.2 (S), Q5.3 (S), R23.1; no longer U3.16 (3V3)
- new net: Q5.5 (D), U3.16 (3V3)
- new net: Q6.3 (D), R22.1
- new net: Q5.4 (G), R22.2, R23.2
- new net: Q6.1 (G), R24.1, R25.2
- new net GNDPWR: Q6.2 (S), R24.2
- new net WLAN_MOD_EN: R25.1
Changed lines of the file:
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@@
 (kicad_sch (version 20211123) (generator eeschema)
   (paper "A3")
+  (junction (at 193.04 60.96) (diameter 0) (color 0 0 0 0)
+  )
   (junction (at 125.73 57.15) (diameter 0) (color 0 0 0 0)
   )
+  (junction (at 203.2 77.47) (diameter 0) (color 0 0 0 0)
+  )
+  (junction (at 209.55 52.07) (diameter 0) (color 0 0 0 0)
+  )
   (junction (at 125.73 59.69) (diameter 0) (color 0 0 0 0)
   )
+  (wire (pts (xy 240.03 86.36) (xy 307.34 86.36))
+    (stroke (width 0) (type default) (color 0 0 0 0))
+  )
   (wire (pts (xy 93.98 110.49) (xy 59.69 110.49))
     (stroke (width 0) (type default) (color 0 0 0 0))
@@
     (stroke (width 0) (type default) (color 0 0 0 0))
   )
-  (wire (pts (xy 125.73 31.75) (xy 125.73 52.07))
+  (wire (pts (xy 203.2 77.47) (xy 200.66 77.47))
     (stroke (width 0) (type default) (color 0 0 0 0))
   )
@@
     (stroke (width 0) (type default) (color 0 0 0 0))
   )
+  (wire (pts (xy 203.2 77.47) (xy 203.2 81.28))
+    (stroke (width 0) (type default) (color 0 0 0 0))
+  )
   (wire (pts (xy 125.73 54.61) (xy 125.73 57.15))
     (stroke (width 0) (type default) (color 0 0 0 0))
   )
+  (wire (pts (xy 193.04 82.55) (xy 193.04 92.71))
+    (stroke (width 0) (type default) (color 0 0 0 0))
+  )
   (wire (pts (xy 120.65 77.47) (xy 154.94 77.47))
     (stroke (width 0) (type default) (color 0 0 0 0))
   )
+  (wire (pts (xy 209.55 49.53) (xy 209.55 52.07))
+    (stroke (width 0) (type default) (color 0 0 0 0))
+  )
+  (wire (pts (xy 198.12 60.96) (xy 193.04 60.96))
+    (stroke (width 0) (type default) (color 0 0 0 0))
+  )
+  (wire (pts (xy 193.04 60.96) (xy 193.04 62.23))
+    (stroke (width 0) (type default) (color 0 0 0 0))
+  )
   (wire (pts (xy 59.69 100.33) (xy 67.31 100.33))
     (stroke (width 0) (type default) (color 0 0 0 0))
@@
     (stroke (width 0) (type default) (color 0 0 0 0))
   )
-  (wire (pts (xy 120.65 52.07) (xy 125.73 52.07))
+  (wire (pts (xy 193.04 69.85) (xy 193.04 72.39))
+    (stroke (width 0) (type default) (color 0 0 0 0))
+  )
+  (wire (pts (xy 207.01 77.47) (xy 203.2 77.47))
+    (stroke (width 0) (type default) (color 0 0 0 0))
+  )
+  (wire (pts (xy 209.55 52.07) (xy 209.55 60.96))
+    (stroke (width 0) (type default) (color 0 0 0 0))
+  )
+  (wire (pts (xy 203.2 88.9) (xy 203.2 92.71))
+    (stroke (width 0) (type default) (color 0 0 0 0))
+  )
+  (wire (pts (xy 193.04 59.69) (xy 193.04 60.96))
+    (stroke (width 0) (type default) (color 0 0 0 0))
+  )
+  (wire (pts (xy 120.65 52.07) (xy 187.96 52.07))
+    (stroke (width 0) (type default) (color 0 0 0 0))
+  )
+  (wire (pts (xy 240.03 77.47) (xy 240.03 86.36))
     (stroke (width 0) (type default) (color 0 0 0 0))
   )
@@
     (stroke (width 0) (type default) (color 0 0 0 0))
   )
+  (wire (pts (xy 214.63 77.47) (xy 240.03 77.47))
+    (stroke (width 0) (type default) (color 0 0 0 0))
+  )
   (wire (pts (xy 120.65 80.01) (xy 154.94 80.01))
     (stroke (width 0) (type default) (color 0 0 0 0))
   )
+  (wire (pts (xy 209.55 52.07) (xy 198.12 52.07))
+    (stroke (width 0) (type default) (color 0 0 0 0))
+  )
   (wire (pts (xy 120.65 59.69) (xy 125.73 59.69))
+    (stroke (width 0) (type default) (color 0 0 0 0))
+  )
+  (wire (pts (xy 205.74 60.96) (xy 209.55 60.96))
     (stroke (width 0) (type default) (color 0 0 0 0))
   )
   (hierarchical_label "UART_0_XDIR" (shape input) (at 59.69 110.49 180)
     (effects (font (size 1.27 1.27)) (justify right))
+  )
+  (hierarchical_label "WLAN_MOD_EN" (shape input) (at 307.34 86.36 0)
+    (effects (font (size 1.27 1.27)) (justify left))
   )
   (hierarchical_label "UART_0_XCK" (shape bidirectional) (at 59.69 100.33 180)
@@
     (pin "9")
   )
+  (symbol (lib_id "Device:R") (at 193.04 66.04 0) (mirror x) (unit 1)
+    (in_bom yes) (on_board yes) (fields_autoplaced)
+    (property "Reference" "R22" (id 0) (at 190.5 64.7699 0)
+      (effects (font (size 1.27 1.27)) (justify right))
+    )
+    (property "Value" "1K" (id 1) (at 190.5 67.3099 0)
+      (effects (font (size 1.27 1.27)) (justify right))
+    )
+    (property "Footprint" "Resistor_SMD:R_0603_1608Metric" (id 2) (at 191.262 66.04 90)
+      (effects (font (size 1.27 1.27)) hide)
+    )
+    (property "Datasheet" "~" (id 3) (at 193.04 66.04 0)
+      (effects (font (size 1.27 1.27)) hide)
+    )
+    (pin "1")
+    (pin "2")
+  )
   (symbol (lib_id "power:GND") (at 125.73 116.84 0) (unit 1)
     (in_bom yes) (on_board yes) (fields_autoplaced)
@@
     (pin "1")
   )
-  (symbol (lib_id "power:+3.3V") (at 125.73 31.75 0) (unit 1)
-    (in_bom yes) (on_board yes) (fields_autoplaced)
-    (property "Reference" "#PWR0130" (id 0) (at 125.73 35.56 0)
-      (effects (font (size 1.27 1.27)) hide)
-    )
-    (property "Value" "+3.3V" (id 1) (at 125.73 26.67 0))
-    (property "Footprint" "" (id 2) (at 125.73 31.75 0)
-      (effects (font (size 1.27 1.27)) hide)
-    )
-    (property "Datasheet" "" (id 3) (at 125.73 31.75 0)
-      (effects (font (size 1.27 1.27)) hide)
-    )
-    (pin "1")
+  (symbol (lib_id "Transistor_FET:Si7141DP") (at 193.04 54.61 90) (unit 1)
+    (in_bom yes) (on_board yes) (fields_autoplaced)
+    (property "Reference" "Q5" (id 0) (at 193.04 44.45 90))
+    (property "Value" "Si7141DP" (id 1) (at 193.04 46.99 90))
+    (property "Footprint" "Package_SO:PowerPAK_SO-8_Single" (id 2) (at 194.945 49.53 0)
+      (effects (font (size 1.27 1.27) italic) (justify left) hide)
+    )
+    (property "Datasheet" "https://www.vishay.com/docs/65596/si7141dp.pdf" (id 3) (at 193.04 54.61 0)
+      (effects (font (size 1.27 1.27)) (justify left) hide)
+    )
+    (pin "1")
+    (pin "2")
+    (pin "3")
+    (pin "4")
+    (pin "5")
+  )
+  (symbol (lib_id "power:GNDPWR") (at 193.04 92.71 0) (mirror y) (unit 1)
+    (in_bom yes) (on_board yes) (fields_autoplaced)
+    (property "Reference" "#PWR035" (id 0) (at 193.04 97.79 0)
+      (effects (font (size 1.27 1.27)) hide)
+    )
+    (property "Value" "GNDPWR" (id 1) (at 193.167 97.79 0))
+    (property "Footprint" "" (id 2) (at 193.04 93.98 0)
+      (effects (font (size 1.27 1.27)) hide)
+    )
+    (property "Datasheet" "" (id 3) (at 193.04 93.98 0)
+      (effects (font (size 1.27 1.27)) hide)
+    )
+    (pin "1")
+  )
+  (symbol (lib_id "Device:R") (at 201.93 60.96 270) (mirror x) (unit 1)
+    (in_bom yes) (on_board yes) (fields_autoplaced)
+    (property "Reference" "R23" (id 0) (at 201.93 54.61 90))
+    (property "Value" "100k" (id 1) (at 201.93 57.15 90))
+    (property "Footprint" "Resistor_SMD:R_0603_1608Metric" (id 2) (at 201.93 62.738 90)
+      (effects (font (size 1.27 1.27)) hide)
+    )
+    (property "Datasheet" "~" (id 3) (at 201.93 60.96 0)
+      (effects (font (size 1.27 1.27)) hide)
+    )
+    (pin "1")
+    (pin "2")
+  )
+  (symbol (lib_id "Device:R") (at 203.2 85.09 0) (mirror y) (unit 1)
+    (in_bom yes) (on_board yes) (fields_autoplaced)
+    (property "Reference" "R24" (id 0) (at 200.66 83.8199 0)
+      (effects (font (size 1.27 1.27)) (justify left))
+    )
+    (property "Value" "1M" (id 1) (at 200.66 86.3599 0)
+      (effects (font (size 1.27 1.27)) (justify left))
+    )
+    (property "Footprint" "Resistor_SMD:R_0603_1608Metric" (id 2) (at 204.978 85.09 90)
+      (effects (font (size 1.27 1.27)) hide)
+    )
+    (property "Datasheet" "~" (id 3) (at 203.2 85.09 0)
+      (effects (font (size 1.27 1.27)) hide)
+    )
+    (pin "1")
+    (pin "2")
+  )
+  (symbol (lib_id "Device:R") (at 210.82 77.47 270) (mirror x) (unit 1)
+    (in_bom yes) (on_board yes) (fields_autoplaced)
+    (property "Reference" "R25" (id 0) (at 210.82 71.12 90))
+    (property "Value" "100R" (id 1) (at 210.82 73.66 90))
+    (property "Footprint" "Resistor_SMD:R_0603_1608Metric" (id 2) (at 210.82 79.248 90)
+      (effects (font (size 1.27 1.27)) hide)
+    )
+    (property "Datasheet" "~" (id 3) (at 210.82 77.47 0)
+      (effects (font (size 1.27 1.27)) hide)
+    )
+    (pin "1")
+    (pin "2")
+  )
+  (symbol (lib_id "power:GNDPWR") (at 203.2 92.71 0) (mirror y) (unit 1)
+    (in_bom yes) (on_board yes) (fields_autoplaced)
+    (property "Reference" "#PWR036" (id 0) (at 203.2 97.79 0)
+      (effects (font (size 1.27 1.27)) hide)
+    )
+    (property "Value" "GNDPWR" (id 1) (at 203.327 97.79 0))
+    (property "Footprint" "" (id 2) (at 203.2 93.98 0)
+      (effects (font (size 1.27 1.27)) hide)
+    )
+    (property "Datasheet" "" (id 3) (at 203.2 93.98 0)
+      (effects (font (size 1.27 1.27)) hide)
+    )
+    (pin "1")
+  )
+  (symbol (lib_id "power:+3.3V") (at 209.55 49.53 0) (unit 1)
+    (in_bom yes) (on_board yes) (fields_autoplaced)
+    (property "Reference" "#PWR0130" (id 0) (at 209.55 53.34 0)
+      (effects (font (size 1.27 1.27)) hide)
+    )
+    (property "Value" "+3.3V" (id 1) (at 209.55 44.45 0))
+    (property "Footprint" "" (id 2) (at 209.55 49.53 0)
+      (effects (font (size 1.27 1.27)) hide)
+    )
+    (property "Datasheet" "" (id 3) (at 209.55 49.53 0)
+      (effects (font (size 1.27 1.27)) hide)
+    )
+    (pin "1")
+  )
+  (symbol (lib_id "Transistor_FET:BSS123") (at 195.58 77.47 0) (mirror y) (unit 1)
+    (in_bom yes) (on_board yes) (fields_autoplaced)
+    (property "Reference" "Q6" (id 0) (at 189.23 76.1999 0)
+      (effects (font (size 1.27 1.27)) (justify left))
+    )
+    (property "Value" "BSS123" (id 1) (at 189.23 78.7399 0)
+      (effects (font (size 1.27 1.27)) (justify left))
+    )
+    (property "Footprint" "Package_TO_SOT_SMD:SOT-23" (id 2) (at 190.5 79.375 0)
+      (effects (font (size 1.27 1.27) italic) (justify left) hide)
+    )
+    (property "Datasheet" "http://www.diodes.com/assets/Datasheets/ds30366.pdf" (id 3) (at 195.58 77.47 0)
+      (effects (font (size 1.27 1.27)) (justify left) hide)
+    )
+    (pin "1")
+    (pin "2")
+    (pin "3")
   )
 )
