File: Hardware/KiCad/Perimeter Sender/Perimeter Sender/POWER_OUTPUT.kicad_sch (KiCad schematic)
At the start: 6 parts, among them U2 INA233, U4 L298N

Commit message: Redesign: - Controller - I2C pinning geändert - uvm
Parts:
- added C5 (x2): 100n, Capacitor_SMD:C_0603_1608Metric, symbol Device:C
- added C5: 1uF, Capacitor_SMD:C_0603_1608Metric, symbol Device:C
Connections:
- net +5V: now also C5.1, C5.1; no longer U2.6 (VS)
- new net +3.3V: C5.1, U2.6 (VS)
- new net GND: C5.2, C5.2, C5.2
